Commit message: Updated description to get the meshes working

File: ros2_ws/src/robot_description/urdf/robot_parts/carcaca.xacro (robot description, xacro)
@@ -21,5 +21,5 @@
                 <origin rpy="0  0  3.14" xyz="0  0  0.0118" />
                 <geometry>
-                    <mesh filename="package://robot_description/models/laser_robot/meshes/carcaca.dae" scale="1 1 1" />
+                    <mesh filename="$(find robot_description)/models/laser_robot/meshes/carcaca.dae" scale="1 1 1" />
                 </geometry>
             </collision>
@@ -27,5 +27,5 @@
                 <origin rpy="0  0  3.14" xyz="0  0  0.0118" />
                 <geometry>
-                    <mesh filename="package://robot_description/models/laser_robot/meshes/carcaca.dae" scale="1 1 1" />
+                    <mesh filename="$(find robot_description)/models/laser_robot/meshes/carcaca.dae" scale="1 1 1" />
                 </geometry>
             </visual>

File: ros2_ws/src/robot_description/urdf/robot_parts/omni_wheel.xacro (robot description, xacro)
@@ -24,5 +24,5 @@
                 <origin rpy="0 0 0" xyz="0 0 0" />
                 <geometry>
-                    <mesh filename="package://robot_description/models/laser_robot/omni_wheel/meshes/roda_omni.obj" scale="1 1 1" />
+                    <mesh filename="$(find robot_description)/models/laser_robot/omni_wheel/meshes/roda_omni.obj" scale="1 1 1" />
                 </geometry>
             </collision>
@@ -30,5 +30,5 @@
                 <origin rpy="0 0 0" xyz="0 0 0" />
                 <geometry>
-                    <mesh filename="package://robot_description/models/laser_robot/omni_wheel/meshes/roda_omni.obj" scale="1 1 1" />
+                    <mesh filename="$(find robot_description)/models/laser_robot/omni_wheel/meshes/roda_omni.obj" scale="1 1 1" />
                 </geometry>
             </visual>

File: ros2_ws/src/robot_description/urdf/robot_parts/piston.xacro (robot description, xacro)
@@ -27,5 +27,5 @@
                 <origin rpy="0  0  0" xyz="0 0 0" />
                 <geometry>
-                    <mesh filename="package://robot_description/models/laser_robot/meshes/piston.dae" scale="1 1 1" />
+                    <mesh filename="$(find robot_description)/models/laser_robot/meshes/piston.dae" scale="1 1 1" />
                 </geometry>
             </collision>
@@ -33,5 +33,5 @@
                 <origin rpy="0  0  0" xyz="0 0 0" />
                 <geometry>
-                    <mesh filename="package://robot_description/models/laser_robot/meshes/piston.dae" scale="1 1 1" />
+                    <mesh filename="$(find robot_description)/models/laser_robot/meshes/piston.dae" scale="1 1 1" />
                 </geometry>
             </visual>

File: ros2_ws/src/robot_description/urdf/robot_parts/traction_wheel.xacro (robot description, xacro)
@@ -30,5 +30,5 @@
                 <origin rpy="0 0 0" xyz="0 0 0" />
                 <geometry>
-                    <mesh filename="package://robot_description/models/laser_robot/wheel/meshes/roda.obj" scale="1 1 1" />
+                    <mesh filename="$(find robot_description)/models/laser_robot/wheel/meshes/roda.obj" scale="1 1 1" />
                 </geometry>
             </collision>
@@ -36,5 +36,5 @@
                 <origin rpy="0 0 0" xyz="0 0 0" />
                 <geometry>
-                    <mesh filename="package://robot_description/models/laser_robot/wheel/meshes/roda.obj" scale="1 1 1" />
+                    <mesh filename="$(find robot_description)/models/laser_robot/wheel/meshes/roda.obj" scale="1 1 1" />
                 </geometry>
             </visual>

File: ros2_ws/src/robot_description/urdf/robot_parts/tray.xacro (robot description, xacro)
@@ -26,5 +26,5 @@
                 <origin rpy="0 0 0" xyz="0 0 0" />
                 <geometry>
-                    <mesh filename="package://robot_description/models/laser_robot/meshes/tray.dae" scale="1 1 1" />
+                    <mesh filename="$(find robot_description)/models/laser_robot/meshes/tray.dae" scale="1 1 1" />
                 </geometry>
             </collision>
@@ -32,5 +32,5 @@
                 <origin rpy="0 0 0" xyz="0 0 0" />
                 <geometry>
-                    <mesh filename="package://robot_description/models/laser_robot/meshes/tray.dae" scale="1 1 1" />
+                    <mesh filename="$(find robot_description)/models/laser_robot/meshes/tray.dae" scale="1 1 1" />
                 </geometry>
             </visual>

File: ros2_ws/src/robot_description/urdf/sensors/camera.xacro (robot description, xacro)
@@ -53,5 +53,5 @@
             <origin rpy="0 0 0" xyz="0 0 0" />
             <geometry>
-                <mesh filename="package://robot_description/models/laser_robot/camera/meshes/camera.obj" scale="0.5 0.5 0.5" />
+                <mesh filename="$(find robot_description)/models/laser_robot/camera/meshes/camera.obj" scale="0.5 0.5 0.5" />
             </geometry>
         </collision>
@@ -59,5 +59,5 @@
             <origin rpy="0 0 1.57" xyz="0 0 0" />
             <geometry>
-                <mesh filename="package://robot_description/models/laser_robot/camera/meshes/camera.obj" scale="0.5 0.5 0.5" />
+                <mesh filename="$(find robot_description)/models/laser_robot/camera/meshes/camera.obj" scale="0.5 0.5 0.5" />
             </geometry>
         </visual>

File: ros2_ws/src/robot_description/urdf/sensors/lidar.xacro (robot description, xacro)
@@ -30,5 +30,5 @@
         </noise>
       </ray>
-      <plugin name="gazebo_ros_head_hokuyo_controller" filename="libgazebo_ros_laser.so">
+      <plugin name="gazebo_ros_head_hokuyo_controller" filename="libgazebo_ros_ray_sensor.so">
         <topicName>/my_robot/laser/scan</topicName>
         <frameName>lidar</frameName>
@@ -50,5 +50,5 @@
       <origin rpy="0 0 0" xyz="0 0 0" />
       <geometry>
-        <mesh filename="package://robot_description/models/laser_robot/lidar/meshes/lidar.obj" scale="0.5 0.5 0.5" />
+        <mesh filename="$(find robot_description)/models/laser_robot/lidar/meshes/lidar.obj" scale="0.5 0.5 0.5" />
       </geometry>
     </collision>
@@ -56,5 +56,5 @@
       <origin rpy="0 1.57 1.57" xyz="0 0 0" />
       <geometry>
-        <mesh filename="package://robot_description/models/laser_robot/lidar/meshes/lidar.obj" scale="0.5 0.5 0.5" />
+        <mesh filename="$(find robot_description)/models/laser_robot/lidar/meshes/lidar.obj" scale="0.5 0.5 0.5" />
       </geometry>
     </visual>

File: ros2_ws/src/robot_description/urdf/sensors/rplidar.xacro (robot description, xacro)
@@ -30,5 +30,5 @@
         </noise>
       </ray>
-      <plugin name="gazebo_ros_head_hokuyo_controller" filename="libgazebo_ros_laser.so">
+      <plugin name="gazebo_ros_head_hokuyo_controllerrp" filename="libgazebo_ros_ray_sensor.so">
         <topicName>/my_robot/rplidar/laser/scan</topicName>
         <frameName>rplidar</frameName>
@@ -50,5 +50,5 @@
       <origin rpy="0 0 1.20" xyz="-0.03 0.02 -0.02" />
       <geometry>
-        <mesh filename="package://robot_description/models/laser_robot/meshes/rplidar.dae" scale="0.7 0.7 0.7" />
+        <mesh filename="$(find robot_description)/models/laser_robot/meshes/rplidar.dae" scale="0.7 0.7 0.7" />
       </geometry>
     </collision>
@@ -56,5 +56,5 @@
       <origin rpy="0 0 1.20" xyz="-0.03 0.02 -0.02" />
       <geometry>
-        <mesh filename="package://robot_description/models/laser_robot/meshes/rplidar.dae" scale="0.7 0.7 0.7" />
+        <mesh filename="$(find robot_description)/models/laser_robot/meshes/rplidar.dae" scale="0.7 0.7 0.7" />
       </geometry>
     </visual>
