Commit message: Change package name from articubot_one to warehouse_robot

File: ros2_ws/src/articubot_one/description/ros2_control.xacro (robot description, xacro)
@@ -56,6 +56,6 @@
     <gazebo>
         <plugin name="gazebo_ros2_control" filename="libgazebo_ros2_control.so">
-            <parameters>$(find articubot_one)/config/my_controllers.yaml</parameters>
-            <parameters>$(find articubot_one)/config/gaz_ros2_ctl_use_sim.yaml</parameters>
+            <parameters>$(find warehouse_robot)/config/my_controllers.yaml</parameters>
+            <parameters>$(find warehouse_robot)/config/gaz_ros2_ctl_use_sim.yaml</parameters>
         </plugin>
     </gazebo>

File: ros2_ws/src/articubot_one/urdf/robot.urdf.xacro (robot description, xacro)
@@ -2,11 +2,11 @@
 <robot name="my_robot" xmlns:xacro="http://www.ros.org/wiki/xacro">
   <!--=========================== PLUGINS ===========================-->
-  <xacro:include filename="$(find articubot_one)/urdf/ros2_control.xacro" />
+  <xacro:include filename="$(find warehouse_robot)/urdf/ros2_control.xacro" />
   <!--=========================== ROBOT PARTS ===========================-->
-  <xacro:include filename="$(find articubot_one)/urdf/robot_parts/carcaca.xacro" />
-  <xacro:include filename="$(find articubot_one)/urdf/robot_parts/traction_wheel.xacro" />
-  <xacro:include filename="$(find articubot_one)/urdf/robot_parts/tray.xacro" />
-  <xacro:include filename="$(find articubot_one)/urdf/robot_parts/piston.xacro" />
-  <xacro:include filename="$(find articubot_one)/urdf/robot_parts/omni_wheel.xacro" />
+  <xacro:include filename="$(find warehouse_robot)/urdf/robot_parts/carcaca.xacro" />
+  <xacro:include filename="$(find warehouse_robot)/urdf/robot_parts/traction_wheel.xacro" />
+  <xacro:include filename="$(find warehouse_robot)/urdf/robot_parts/tray.xacro" />
+  <xacro:include filename="$(find warehouse_robot)/urdf/robot_parts/piston.xacro" />
+  <xacro:include filename="$(find warehouse_robot)/urdf/robot_parts/omni_wheel.xacro" />
   <!--=========================== SENSORS ===========================-->
   <!-- <xacro:arg name="sensor_imu" default="true" /> -->
@@ -15,14 +15,14 @@
   <xacro:arg name="sensor_camera" default="true" />
   <!-- <xacro:if value="$(arg sensor_imu)">
-    <xacro:include filename="$(find articubot_one)/urdf/sensors/imu.xacro" />
+    <xacro:include filename="$(find warehouse_robot)/urdf/sensors/imu.xacro" />
   </xacro:if> -->
   <xacro:if value="$(arg sensor_lidar)">
-    <xacro:include filename="$(find articubot_one)/urdf/sensors/lidar.xacro" />
+    <xacro:include filename="$(find warehouse_robot)/urdf/sensors/lidar.xacro" />
   </xacro:if>
   <!-- <xacro:if value="$(arg sensor_rplidar)">
-    <xacro:include filename="$(find articubot_one)/urdf/sensors/rplidar.xacro" />
+    <xacro:include filename="$(find warehouse_robot)/urdf/sensors/rplidar.xacro" />
   </xacro:if> -->
   <xacro:if value="$(arg sensor_camera)">
-    <xacro:include filename="$(find articubot_one)/urdf/sensors/camera.xacro" />
+    <xacro:include filename="$(find warehouse_robot)/urdf/sensors/camera.xacro" />
   </xacro:if>
 </robot>

File: ros2_ws/src/articubot_one/urdf/robot_parts/carcaca.xacro (robot description, xacro)
@@ -21,5 +21,5 @@
                 <origin rpy="0  0  3.14" xyz="0  0  0.0118" />
                 <geometry>
-                    <mesh filename="$(find articubot_one)/models/laser_robot/meshes/carcaca.dae" scale="1 1 1" />
+                    <mesh filename="$(find warehouse_robot)/models/laser_robot/meshes/carcaca.dae" scale="1 1 1" />
                 </geometry>
             </collision>
@@ -27,5 +27,5 @@
                 <origin rpy="0  0  3.14" xyz="0  0  0.0118" />
                 <geometry>
-                    <mesh filename="$(find articubot_one)/models/laser_robot/meshes/carcaca.dae" scale="1 1 1" />
+                    <mesh filename="$(find warehouse_robot)/models/laser_robot/meshes/carcaca.dae" scale="1 1 1" />
                 </geometry>
             </visual>

File: ros2_ws/src/articubot_one/urdf/robot_parts/omni_wheel.xacro (robot description, xacro)
@@ -24,5 +24,5 @@
                 <origin rpy="0 0 0" xyz="0 0 0" />
                 <geometry>
-                    <mesh filename="$(find articubot_one)/models/laser_robot/omni_wheel/meshes/roda_omni.obj" scale="1 1 1" />
+                    <mesh filename="$(find warehouse_robot)/models/laser_robot/omni_wheel/meshes/roda_omni.obj" scale="1 1 1" />
                 </geometry>
             </collision>
@@ -30,5 +30,5 @@
                 <origin rpy="0 0 0" xyz="0 0 0" />
                 <geometry>
-                    <mesh filename="$(find articubot_one)/models/laser_robot/omni_wheel/meshes/roda_omni.obj" scale="1 1 1" />
+                    <mesh filename="$(find warehouse_robot)/models/laser_robot/omni_wheel/meshes/roda_omni.obj" scale="1 1 1" />
                 </geometry>
             </visual>

File: ros2_ws/src/articubot_one/urdf/robot_parts/piston.xacro (robot description, xacro)
@@ -27,5 +27,5 @@
                 <origin rpy="0  0  0" xyz="0 0 0" />
                 <geometry>
-                    <mesh filename="$(find articubot_one)/models/laser_robot/meshes/piston.dae" scale="1 1 1" />
+                    <mesh filename="$(find warehouse_robot)/models/laser_robot/meshes/piston.dae" scale="1 1 1" />
                 </geometry>
             </collision>
@@ -33,5 +33,5 @@
                 <origin rpy="0  0  0" xyz="0 0 0" />
                 <geometry>
-                    <mesh filename="$(find articubot_one)/models/laser_robot/meshes/piston.dae" scale="1 1 1" />
+                    <mesh filename="$(find warehouse_robot)/models/laser_robot/meshes/piston.dae" scale="1 1 1" />
                 </geometry>
             </visual>

File: ros2_ws/src/articubot_one/urdf/robot_parts/traction_wheel.xacro (robot description, xacro)
@@ -30,5 +30,5 @@
                 <origin rpy="0 0 0" xyz="0 0 0" />
                 <geometry>
-                    <mesh filename="$(find articubot_one)/models/laser_robot/wheel/meshes/roda.obj" scale="1 1 1" />
+                    <mesh filename="$(find warehouse_robot)/models/laser_robot/wheel/meshes/roda.obj" scale="1 1 1" />
                 </geometry>
             </collision>
@@ -36,5 +36,5 @@
                 <origin rpy="0 0 0" xyz="0 0 0" />
                 <geometry>
-                    <mesh filename="$(find articubot_one)/models/laser_robot/wheel/meshes/roda.obj" scale="1 1 1" />
+                    <mesh filename="$(find warehouse_robot)/models/laser_robot/wheel/meshes/roda.obj" scale="1 1 1" />
                 </geometry>
             </visual>

File: ros2_ws/src/articubot_one/urdf/robot_parts/tray.xacro (robot description, xacro)
@@ -26,5 +26,5 @@
                 <origin rpy="0 0 0" xyz="0 0 0" />
                 <geometry>
-                    <mesh filename="$(find articubot_one)/models/laser_robot/meshes/tray.dae" scale="1 1 1" />
+                    <mesh filename="$(find warehouse_robot)/models/laser_robot/meshes/tray.dae" scale="1 1 1" />
                 </geometry>
             </collision>
@@ -32,5 +32,5 @@
                 <origin rpy="0 0 0" xyz="0 0 0" />
                 <geometry>
-                    <mesh filename="$(find articubot_one)/models/laser_robot/meshes/tray.dae" scale="1 1 1" />
+                    <mesh filename="$(find warehouse_robot)/models/laser_robot/meshes/tray.dae" scale="1 1 1" />
                 </geometry>
             </visual>

File: ros2_ws/src/articubot_one/urdf/sensors/camera.xacro (robot description, xacro)
@@ -53,5 +53,5 @@
             <origin rpy="0 0 0" xyz="0 0 0" />
             <geometry>
-                <mesh filename="$(find articubot_one)/models/laser_robot/camera/meshes/camera.obj" scale="0.5 0.5 0.5" />
+                <mesh filename="$(find warehouse_robot)/models/laser_robot/camera/meshes/camera.obj" scale="0.5 0.5 0.5" />
             </geometry>
         </collision>
@@ -59,5 +59,5 @@
             <origin rpy="0 0 1.57" xyz="0 0 0" />
             <geometry>
-                <mesh filename="$(find articubot_one)/models/laser_robot/camera/meshes/camera.obj" scale="0.5 0.5 0.5" />
+                <mesh filename="$(find warehouse_robot)/models/laser_robot/camera/meshes/camera.obj" scale="0.5 0.5 0.5" />
             </geometry>
         </visual>

File: ros2_ws/src/articubot_one/urdf/sensors/lidar.xacro (robot description, xacro)
@@ -53,5 +53,5 @@
       <origin rpy="0 0 0" xyz="0 0 0" />
       <geometry>
-        <mesh filename="$(find articubot_one)/models/laser_robot/lidar/meshes/lidar.obj" scale="0.5 0.5 0.5" />
+        <mesh filename="$(find warehouse_robot)/models/laser_robot/lidar/meshes/lidar.obj" scale="0.5 0.5 0.5" />
       </geometry>
     </collision>
@@ -59,5 +59,5 @@
       <origin rpy="0 1.57 1.57" xyz="0 0 0" />
       <geometry>
-        <mesh filename="$(find articubot_one)/models/laser_robot/lidar/meshes/lidar.obj" scale="0.5 0.5 0.5" />
+        <mesh filename="$(find warehouse_robot)/models/laser_robot/lidar/meshes/lidar.obj" scale="0.5 0.5 0.5" />
       </geometry>
     </visual>

File: ros2_ws/src/articubot_one/urdf/sensors/rplidar.xacro (robot description, xacro)
@@ -50,5 +50,5 @@
       <origin rpy="0 0 1.20" xyz="-0.03 0.02 -0.02" />
       <geometry>
-        <mesh filename="$(find articubot_one)/models/laser_robot/meshes/rplidar.dae" scale="0.7 0.7 0.7" />
+        <mesh filename="$(find warehouse_robot)/models/laser_robot/meshes/rplidar.dae" scale="0.7 0.7 0.7" />
       </geometry>
     </collision>
@@ -56,5 +56,5 @@
       <origin rpy="0 0 1.20" xyz="-0.03 0.02 -0.02" />
       <geometry>
-        <mesh filename="$(find articubot_one)/models/laser_robot/meshes/rplidar.dae" scale="0.7 0.7 0.7" />
+        <mesh filename="$(find warehouse_robot)/models/laser_robot/meshes/rplidar.dae" scale="0.7 0.7 0.7" />
       </geometry>
     </visual>
