Commit message: Camera now points at the ground

File: ros2_ws/src/warehouse_robot/description/camera.xacro (robot description, xacro)
@@ -4,5 +4,5 @@
         <parent link="chassis"/>
         <child link="camera_link"/>
-        <origin xyz="0.276 0 0.181" rpy="0 0.18 0"/>
+        <origin xyz="0.7 0 0.181" rpy="0 1.57 0"/>
     </joint>
     <link name="camera_link">
