Commit message: Updated remaining joint_piston names and changed piston controller name to piston_cont

File: ros2_ws/src/warehouse_robot/description/gazebo_control.xacro (robot description, xacro)
@@ -21,5 +21,5 @@
     <gazebo>
         <plugin name="joint_state_publisher" filename="libgazebo_ros_joint_state_publisher.so">
-          <jointName>piston_joint, tray_joint</jointName>
+          <jointName>joint_piston, tray_joint</jointName>
         </plugin>
       </gazebo>

File: ros2_ws/src/warehouse_robot/description/robot_core.xacro (robot description, xacro)
@@ -157,5 +157,5 @@
     </gazebo>
     <!-- Piston -->
-    <joint name="piston_joint" type="prismatic">
+    <joint name="joint_piston" type="prismatic">
         <parent link="chassis"/>
         <child link="piston"/>

File: ros2_ws/src/warehouse_robot/description/ros2_control.xacro (robot description, xacro)
@@ -52,5 +52,5 @@
                 <state_interface name="position"/>
             </joint>
-            <joint name="piston_joint">
+            <joint name="joint_piston">
                 <command_interface name="position">
                     <param name="min">-10</param>

File: ros2_ws/src/warehouse_robot/urdf/ros2_control.xacro (robot description, xacro)
@@ -21,5 +21,5 @@
                 <state_interface name="position"/>
             </joint>
-            <joint name="piston_joint">
+            <joint name="joint_piston">
                 <command_interface name="position">
                     <param name="min">-10</param>
@@ -37,5 +37,5 @@
     <transmission name="tran1">
         <type>transmission_interface/SimpleTransmission</type>
-        <joint name="piston_joint">
+        <joint name="joint_piston">
           <hardwareInterface>hardware_interface/EffortJointInterface</hardwareInterface>
         </joint>
