Commit message: Added position controller for piston joint

File: ros2_ws/src/warehouse_robot/description/ros2_control.xacro (robot description, xacro)
@@ -52,4 +52,11 @@
                 <state_interface name="position"/>
             </joint>
+            <joint name="joint_piston">
+                <command_interface name="position">
+                    <param name="min">-10</param>
+                    <param name="max">10</param>
+                </command_interface>
+                <state_interface name="position"/>
+            </joint>
         </ros2_control>
     </xacro:if>

Commit message: Attempted to get one controller working with multiple robots and namespaces for joints

File: ros2_ws/src/warehouse_robot/description/ros2_control.xacro (robot description, xacro)
@@ -36,5 +36,5 @@
                 <plugin>gazebo_ros2_control/GazeboSystem</plugin>
             </hardware>
-            <joint name="left_wheel_joint">
+            <joint name="$(arg namespace)_left_wheel_joint">
                 <command_interface name="velocity">
                     <param name="min">-10</param>
@@ -44,5 +44,5 @@
                 <state_interface name="position"/>
             </joint>
-            <joint name="right_wheel_joint">
+            <joint name="$(arg namespace)_right_wheel_joint">
                 <command_interface name="velocity">
                     <param name="min">-10</param>
@@ -52,5 +52,5 @@
                 <state_interface name="position"/>
             </joint>
-            <joint name="joint_piston">
+            <joint name="$(arg namespace)_joint_piston">
                 <command_interface name="position">
                     <param name="min">-10</param>

File: ros2_ws/src/warehouse_robot/urdf/robot_1.urdf.xacro (robot description, xacro)
@@ -2,13 +2,13 @@
 <robot name="my_robot_1" xmlns:xacro="http://www.ros.org/wiki/xacro">
   <!--=========================== PLUGINS ===========================-->
-  <xacro:include filename="$(find warehouse_robot)/urdf/ros2_control.xacro" />
+  <xacro:include filename="$(find warehouse_robot)/urdf/ros2_control.xacro" ns="robot_1" />
   <!--=========================== ROBOT PARTS ===========================-->
-  <xacro:include filename="$(find warehouse_robot)/urdf/robot_parts/carcaca.xacro" />
-  <xacro:include filename="$(find warehouse_robot)/urdf/robot_parts/traction_wheel.xacro" />
-  <xacro:include filename="$(find warehouse_robot)/urdf/robot_parts/tray.xacro" />
-  <xacro:include filename="$(find warehouse_robot)/urdf/robot_parts/piston.xacro" />
-  <xacro:include filename="$(find warehouse_robot)/urdf/robot_parts/omni_wheel.xacro" />
+  <xacro:include filename="$(find warehouse_robot)/urdf/robot_parts/carcaca.xacro" ns="robot_1"/>
+  <xacro:include filename="$(find warehouse_robot)/urdf/robot_parts/traction_wheel.xacro" ns="robot_1"/>
+  <xacro:include filename="$(find warehouse_robot)/urdf/robot_parts/tray.xacro" ns="robot_1"/>
+  <xacro:include filename="$(find warehouse_robot)/urdf/robot_parts/piston.xacro" ns="robot_1"/>
+  <xacro:include filename="$(find warehouse_robot)/urdf/robot_parts/omni_wheel.xacro" ns="robot_1"/>
   <!--=========================== SENSORS ===========================-->
-    <xacro:include filename="$(find warehouse_robot)/urdf/sensors/rplidar.xacro" />
-    <xacro:include filename="$(find warehouse_robot)/urdf/sensors/camera.xacro" />
+    <xacro:include filename="$(find warehouse_robot)/urdf/sensors/rplidar.xacro" ns="robot_1"/>
+    <xacro:include filename="$(find warehouse_robot)/urdf/sensors/camera.xacro" ns="robot_1"/>
 </robot>

File: ros2_ws/src/warehouse_robot/urdf/robot_2.urdf.xacro (robot description, xacro)
@@ -2,13 +2,13 @@
 <robot name="my_robot_2" xmlns:xacro="http://www.ros.org/wiki/xacro">
   <!--=========================== PLUGINS ===========================-->
-  <xacro:include filename="$(find warehouse_robot)/urdf/ros2_control.xacro" />
+  <xacro:include filename="$(find warehouse_robot)/urdf/ros2_control.xacro" ns="robot_2"/>
   <!--=========================== ROBOT PARTS ===========================-->
-  <xacro:include filename="$(find warehouse_robot)/urdf/robot_parts/carcaca.xacro" />
-  <xacro:include filename="$(find warehouse_robot)/urdf/robot_parts/traction_wheel.xacro" />
-  <xacro:include filename="$(find warehouse_robot)/urdf/robot_parts/tray.xacro" />
-  <xacro:include filename="$(find warehouse_robot)/urdf/robot_parts/piston.xacro" />
-  <xacro:include filename="$(find warehouse_robot)/urdf/robot_parts/omni_wheel.xacro" />
+  <xacro:include filename="$(find warehouse_robot)/urdf/robot_parts/carcaca.xacro" ns="robot_2"/>
+  <xacro:include filename="$(find warehouse_robot)/urdf/robot_parts/traction_wheel.xacro" ns="robot_2"/>
+  <xacro:include filename="$(find warehouse_robot)/urdf/robot_parts/tray.xacro" ns="robot_2" />
+  <xacro:include filename="$(find warehouse_robot)/urdf/robot_parts/piston.xacro" ns="robot_2"/>
+  <xacro:include filename="$(find warehouse_robot)/urdf/robot_parts/omni_wheel.xacro" ns="robot_2"/>
   <!--=========================== SENSORS ===========================-->
-    <xacro:include filename="$(find warehouse_robot)/urdf/sensors/rplidar.xacro" />
-    <xacro:include filename="$(find warehouse_robot)/urdf/sensors/camera.xacro" />
+    <xacro:include filename="$(find warehouse_robot)/urdf/sensors/rplidar.xacro" ns="robot_2"/>
+    <xacro:include filename="$(find warehouse_robot)/urdf/sensors/camera.xacro" ns="robot_2"/>
 </robot>

File: ros2_ws/src/warehouse_robot/urdf/robot_parts/omni_wheel.xacro (robot description, xacro)
@@ -1,5 +1,5 @@
 <?xml version="1.0"?>
 <robot xmlns:xacro="http://www.ros.org/wiki/xacro">
-    <xacro:macro name="omni_wheel" params="prefix pos_X pos_Y pos_Z pos_r pos_p pos_y">
+    <xacro:macro name="omni_wheel" params="namespace prefix pos_X pos_Y pos_Z pos_r pos_p pos_y">
         <joint name="joint_${prefix}_wheel" type="fixed">
             <parent link="base_link" />

File: ros2_ws/src/warehouse_robot/urdf/robot_parts/piston.xacro (robot description, xacro)
@@ -1,5 +1,5 @@
 <?xml version="1.0"?>
 <robot xmlns:xacro="http://www.ros.org/wiki/xacro">
-    <xacro:macro name="piston" params="prefix">
+    <xacro:macro name="piston" params="namespace prefix">
         <joint name="joint_${prefix}" type="prismatic">
             <parent link="carcaca" />

File: ros2_ws/src/warehouse_robot/urdf/robot_parts/traction_wheel.xacro (robot description, xacro)
@@ -1,5 +1,5 @@
 <?xml version="1.0"?>
 <robot xmlns:xacro="http://www.ros.org/wiki/xacro">
-    <xacro:macro name="traction_wheel" params="prefix pos_X pos_Y pos_Z pos_r pos_p pos_y axis">
+    <xacro:macro name="traction_wheel" params="namespace prefix pos_X pos_Y pos_Z pos_r pos_p pos_y axis">
         <joint name="${prefix}_joint" type="continuous">
             <parent link="base_link" />

File: ros2_ws/src/warehouse_robot/urdf/robot_parts/tray.xacro (robot description, xacro)
@@ -1,5 +1,5 @@
 <?xml version="1.0"?>
 <robot xmlns:xacro="http://www.ros.org/wiki/xacro">
-    <xacro:macro name="tray" params="prefix">
+    <xacro:macro name="tray" params="namespace prefix">
         <joint name="joint_${prefix}" type="continuous">
             <parent link="piston" />
