Commit message: Slightly increase rpi lidar height

File: ros2_ws/src/warehouse_robot/urdf/sensors/rplidar.xacro (robot description, xacro)
@@ -39,5 +39,5 @@
     <parent link="base_link" />
     <child link="rplidar" />
-    <origin rpy="0 0 0" xyz="0.14 -0.17 0.25" />
+    <origin rpy="0 0 0" xyz="0.14 -0.17 0.255" />
   </joint>
   <link name="rplidar">
