Commit message: Updated the wrong file... removed the dup

File: ros2_ws/src/warehouse_robot/urdf/sensors/camera.xacro (robot description, xacro)
@@ -1,9 +1,8 @@
 <?xml version="1.0"?>
 <robot xmlns:xacro="http://www.ros.org/wiki/xacro">
-    <xacro:arg name="camera_1_visual" default="true" />
     <gazebo reference="camera_link">
         <sensor type="camera" name="camera">
             <update_rate>30.0</update_rate>
-            <visualize>$(arg camera_1_visual)</visualize>
+            <visualize>true</visualize>
             <camera name="camera">
                 <horizontal_fov>1.3962634</horizontal_fov>
@@ -41,8 +40,8 @@
     <joint name="camera_joint" type="fixed">
         <parent link="carcaca" />
-        <child link="camera_link" />
+        <child link="camera_link_optical" />
         <origin rpy="0 1.57 0" xyz="0 0 0.0367" />
     </joint>
-    <link name="camera_link">
+    <link name="camera_link_optical">
         <inertial>
             <mass value="0.1" />
@@ -50,5 +49,5 @@
             <inertia ixx="1" ixy="0" ixz="0" iyy="1" iyz="0" izz="1" />
         </inertial>
-        <collision name="camera_link_collision">
+        <collision>
             <origin rpy="0 0 0" xyz="0 0 0" />
             <geometry>
@@ -56,5 +55,5 @@
             </geometry>
         </collision>
-        <visual name="camera_link_visual">
+        <visual>
             <origin rpy="0 0 1.57" xyz="0 0 0" />
             <geometry>

Commit message: Changes to the AprilTag module
- Homogeneous transformations to get the robot pose from the preset tag pose corrected
- homography matrix to pose corrected
- return robot's anular pose added

File: ros2_ws/src/warehouse_robot/urdf/sensors/camera.xacro (robot description, xacro)
@@ -13,6 +13,6 @@
                 </image>
                 <clip>
-                    <near>0.02</near>
-                    <far>300</far>
+                    <near>0.01</near>
+                    <far>500</far>
                 </clip>
                 <!-- <noise>
@@ -23,9 +23,9 @@
             </camera>
             <plugin name="camera_controller" filename="libgazebo_ros_camera.so">
-                <!-- <alwaysOn>true</alwaysOn> -->
+                <alwaysOn>true</alwaysOn>
                 <!-- <updateRate>0.0</updateRate> -->
-                <!-- <cameraName>my_robot/camera1</cameraName> -->
-                <!-- <imageTopicName>image_raw</imageTopicName> -->
-                <!-- <cameraInfoTopicName>camera_info</cameraInfoTopicName> -->
+                <cameraName>camera</cameraName>
+                <imageTopicName>image_raw</imageTopicName>
+                <cameraInfoTopicName>camera_info</cameraInfoTopicName>
                 <frameName>camera_link_optical</frameName>
                 <!-- <hackBaseline>0.07</hackBaseline> -->
@@ -41,5 +41,5 @@
         <parent link="base_link" />
         <child link="camera_link" />
-        <origin rpy="0 1.57 0" xyz="0 0 0.0367" />
+        <origin rpy="0 1.57 0" xyz="0 0 0.045" />
     </joint>
     <joint name="camera_optical_joint" type="fixed">
