Commit message: fix for camera urdf

File: ros2_ws/src/warehouse_robot/urdf/camera.xacro (robot description, xacro)
@@ -1,52 +1,64 @@
 <?xml version="1.0"?>
 <robot xmlns:xacro="http://www.ros.org/wiki/xacro" >
-    <joint name="camera_joint" type="fixed">
-        <parent link="chassis"/>
-        <child link="camera_link"/>
-        <origin xyz="0.276 0 0.181" rpy="0 0.18 0"/>
-    </joint>
-    <link name="camera_link">
-        <visual>
-            <geometry>
-                <box size="0.010 0.03 0.03"/>
-            </geometry>
-            <material name="black"/>
-        </visual>
-        <visual>
-            <origin xyz="0 0 -0.05"/>
-            <geometry>
-                <cylinder radius="0.002" length="0.1"/>
-            </geometry>
-            <material name="black"/>
-        </visual>
-    </link>
-    <joint name="camera_optical_joint" type="fixed">
-        <parent link="camera_link"/>
-        <child link="camera_link_optical"/>
-        <origin xyz="0 0 0" rpy="${-pi/2} 0 ${-pi/2}"/>
-    </joint>
-    <link name="camera_link_optical"></link>
     <gazebo reference="camera_link">
-        <material>Gazebo/Black</material>
-        <sensor name="camera" type="camera">
-            <pose> 0 0 0 0 0 0 </pose>
-            <visualize>true</visualize>
-            <update_rate>10</update_rate>
+        <sensor type="camera" name="camera1">
+            <update_rate>30.0</update_rate>
+            <visualize>$(arg camera_1_visual)</visualize>
             <camera>
-                <horizontal_fov>1.089</horizontal_fov>
+                <horizontal_fov>1.3962634</horizontal_fov>
                 <image>
+                    <width>800</width>
+                    <height>800</height>
                     <format>R8G8B8</format>
-                    <width>640</width>
-                    <height>480</height>
                 </image>
                 <clip>
-                    <near>0.05</near>
-                    <far>8.0</far>
+                    <near>0.02</near>
+                    <far>300</far>
                 </clip>
+                <noise>
+                    <type>gaussian</type>
+                    <mean>0.0</mean>
+                    <stddev>0.007</stddev>
+                </noise>
             </camera>
             <plugin name="camera_controller" filename="libgazebo_ros_camera.so">
-                <frame_name>camera_link_optical</frame_name>
+                <!-- <alwaysOn>true</alwaysOn> -->
+                <!-- <updateRate>0.0</updateRate> -->
+                <!-- <cameraName>my_robot/camera1</cameraName> -->
+                <!-- <imageTopicName>image_raw</imageTopicName> -->
+                <cameraInfoTopicName>camera_info</cameraInfoTopicName>
+                <frameName>camera_link_optical</frameName>
+                <hackBaseline>0.07</hackBaseline>
+                <distortionK1>0.0</distortionK1>
+                <distortionK2>0.0</distortionK2>
+                <distortionK3>0.0</distortionK3>
+                <distortionT1>0.0</distortionT1>
+                <distortionT2>0.0</distortionT2>
             </plugin>
         </sensor>
     </gazebo>
+    <joint name="camera_optical_joint" type="fixed">
+        <parent link="carcaca" />
+        <child link="camera_link_optical" />
+        <origin rpy="0 1.57 0" xyz="0 0 0.0367" />
+    </joint>
+    <link name="camera_link_optical">
+        <inertial>
+            <mass value="0.1" />
+            <origin rpy="0 0 0" xyz="0 0 0" />
+            <inertia ixx="1" ixy="0" ixz="0" iyy="1" iyz="0" izz="1" />
+        </inertial>
+        <collision>
+            <origin rpy="0 0 0" xyz="0 0 0" />
+            <geometry>
+                <mesh filename="$(find warehouse_robot)/models/laser_robot/camera/meshes/camera.obj" scale="0.5 0.5 0.5" />
+            </geometry>
+        </collision>
+        <visual>
+            <origin rpy="0 0 1.57" xyz="0 0 0" />
+            <geometry>
+                <mesh filename="$(find warehouse_robot)/models/laser_robot/camera/meshes/camera.obj" scale="0.5 0.5 0.5" />
+            </geometry>
+        </visual>
+    </link>
 </robot>
