Commit message: Added imu and ekf_filtering

File: ros2_ws/src/warehouse_robot/urdf/gazebo_control.xacro (robot description, xacro)
@@ -3,18 +3,38 @@
     <gazebo>
         <plugin name="diff_drive" filename="libgazebo_ros_diff_drive.so">
-            <!-- Wheel Information -->
-            <left_joint>left_wheel_joint</left_joint>
-            <right_joint>right_wheel_joint</right_joint>
-            <wheel_separation>0.297</wheel_separation>
-            <wheel_diameter>0.066</wheel_diameter>
-            <!-- Limits -->
-            <max_wheel_torque>200</max_wheel_torque>
-            <max_wheel_acceleration>10.0</max_wheel_acceleration>
-            <!-- Output -->
-            <odometry_frame>odom</odometry_frame>
-            <robot_base_frame>base_link</robot_base_frame>
-            <publish_odom>true</publish_odom>
-            <publish_odom_tf>true</publish_odom_tf>
-            <publish_wheel_tf>true</publish_wheel_tf>
+            <!-- Plugin update rate in Hz -->
+            <updateRate>50</updateRate>
+            <!-- Name of left joint, defaults to `left_joint` -->
+            <leftJoint>left_wheel_joint</leftJoint>
+            <!-- Name of right joint, defaults to `right_joint` -->
+            <rightJoint>right_wheel_joint</rightJoint>
+            <!-- The distance from the center of one wheel to the other, in meters, defaults to 0.34
+            m -->
+            <wheelSeparation>0.407</wheelSeparation>
+            <!-- Diameter of the wheels, in meters, defaults to 0.15 m -->
+            <wheelDiameter>0.1016</wheelDiameter>
+            <!-- Wheel acceleration, in rad/s^2, defaults to 0.0 rad/s^2 -->
+            <wheelAcceleration>0</wheelAcceleration>
+            <!-- Maximum torque which the wheels can produce, in Nm, defaults to 5 Nm -->
+            <wheelTorque>3</wheelTorque>
+            <!-- Topic to receive geometry_msgs/Twist message commands, defaults to `cmd_vel` -->
+            <commandTopic>cmd_vel</commandTopic>
+            <!-- Topic to publish nav_msgs/Odometry messages, defaults to `odom` -->
+            <odometryTopic>odom</odometryTopic>
+            <!-- Odometry frame, defaults to `odom` -->
+            <odometryFrame>odom</odometryFrame>
+            <!-- Robot frame to calculate odometry from, defaults to `base_footprint` -->
+            <robotBaseFrame>base_link</robotBaseFrame>
+            <!-- Odometry source, 0 for ENCODER, 1 for WORLD, defaults to WORLD -->
+            <odometrySource>1</odometrySource>
+            <!-- Set to true to publish transforms for the wheel links, defaults to false -->
+            <publishWheelTF>false</publishWheelTF>
+            <!-- Set to true to publish transforms for the odometry, defaults to true -->
+            <publishOdom>true</publishOdom>
+            <!-- Set to true to publish sensor_msgs/JointState on /joint_states for the wheel
+            joints, defaults to false -->
+            <publishWheelJointState>true</publishWheelJointState>
+            <!-- Set to true to swap right and left wheels, defaults to true -->
+            <legacyMode>false</legacyMode>
         </plugin>
     </gazebo>

File: ros2_ws/src/warehouse_robot/urdf/robot.urdf.xacro (robot description, xacro)
@@ -2,5 +2,5 @@
 <robot name="my_robot" xmlns:xacro="http://www.ros.org/wiki/xacro">
   <!--=========================== PLUGINS ===========================-->
-  <xacro:include filename="$(find warehouse_robot)/urdf/ros2_control.xacro" />
+  <!-- <xacro:include filename="$(find warehouse_robot)/urdf/ros2_control.xacro" /> -->
   <!--=========================== ROBOT PARTS ===========================-->
   <xacro:include filename="$(find warehouse_robot)/urdf/robot_parts/carcaca.xacro" />

File: ros2_ws/src/warehouse_robot/urdf/robot_parts/carcaca.xacro (robot description, xacro)
@@ -11,15 +11,21 @@
         </gazebo>
         <joint name="base_footprint_joint" type="fixed">
-            <parent link="base_link"/>
-            <child link="base_footprint"/>
-            <origin xyz="0 0 0" rpy="0 0 0"/>
+            <parent link="base_link" />
+            <child link="base_footprint" />
+            <origin xyz="0 0 0" rpy="0 0 0" />
         </joint>
         <joint name="chassis_joint" type="fixed">
-            <parent link="base_link"/>
-            <child link="${base_link}"/>
-            <origin xyz="0 0 0" rpy="0 0 -1.57"/>
+            <parent link="base_link" />
+            <child link="${base_link}" />
+            <origin xyz="0 0 0" rpy="0 0 -1.57" />
+        </joint>
+        <joint name="imu_joint" type="fixed">
+            <parent link="base_link"></parent>
+            <child link="imu_link"></child>
+            <origin xyz="0 0 0.01"></origin>
         </joint>
         <link name="base_link">
         </link>
+        <link name="imu_link"></link>
         <link name="base_footprint">
         </link>
@@ -29,11 +35,12 @@
                 <origin rpy="0  0  0" xyz="0  0  0.0118" />
                 <inertia ixx="0.019995" ixy="0.0" ixz="0.0"
-                iyy="0.019995" iyz="0.0"
-                izz="0.03675" />
+                    iyy="0.019995" iyz="0.0"
+                    izz="0.03675" />
             </inertial>
             <collision name="${base_link}_collision">
                 <origin rpy="0  0  0" xyz="0  0  0.0118" />
                 <geometry>
-                    <mesh filename="$(find warehouse_robot)/models/laser_robot/meshes/carcaca.dae" scale="1 1 1" />
+                    <mesh filename="$(find warehouse_robot)/models/laser_robot/meshes/carcaca.dae"
+                        scale="1 1 1" />
                 </geometry>
             </collision>
@@ -41,8 +48,76 @@
                 <origin rpy="0  0  0" xyz="0  0  0.0118" />
                 <geometry>
-                    <mesh filename="$(find warehouse_robot)/models/laser_robot/meshes/carcaca.dae" scale="1 1 1" />
+                    <mesh filename="$(find warehouse_robot)/models/laser_robot/meshes/carcaca.dae"
+                        scale="1 1 1" />
                 </geometry>
             </visual>
         </link>
+        <gazebo reference="imu_link">
+            <sensor name="imu_sensor" type="imu">
+                <plugin filename="libgazebo_ros_imu_sensor.so" name="imu_plugin">
+                    <ros>
+                        <remapping>~/out:=imu</remapping>
+                    </ros>
+                    <initial_orientation_as_reference>false</initial_orientation_as_reference>
+                </plugin>
+                <always_on>true</always_on>
+                <update_rate>100</update_rate>
+                <visualize>true</visualize>
+                <imu>
+                    <angular_velocity>
+                        <x>
+                            <noise type="gaussian">
+                                <mean>0.0</mean>
+                                <stddev>2e-4</stddev>
+                                <bias_mean>0.0000075</bias_mean>
+                                <bias_stddev>0.0000008</bias_stddev>
+                            </noise>
+                        </x>
+                        <y>
+                            <noise type="gaussian">
+                                <mean>0.0</mean>
+                                <stddev>2e-4</stddev>
+                                <bias_mean>0.0000075</bias_mean>
+                                <bias_stddev>0.0000008</bias_stddev>
+                            </noise>
+                        </y>
+                        <z>
+                            <noise type="gaussian">
+                                <mean>0.0</mean>
+                                <stddev>2e-4</stddev>
+                                <bias_mean>0.0000075</bias_mean>
+                                <bias_stddev>0.0000008</bias_stddev>
+                            </noise>
+                        </z>
+                    </angular_velocity>
+                    <linear_acceleration>
+                        <x>
+                            <noise type="gaussian">
+                                <mean>0.0</mean>
+                                <stddev>1.7e-2</stddev>
+                                <bias_mean>0.1</bias_mean>
+                                <bias_stddev>0.001</bias_stddev>
+                            </noise>
+                        </x>
+                        <y>
+                            <noise type="gaussian">
+                                <mean>0.0</mean>
+                                <stddev>1.7e-2</stddev>
+                                <bias_mean>0.1</bias_mean>
+                                <bias_stddev>0.001</bias_stddev>
+                            </noise>
+                        </y>
+                        <z>
+                            <noise type="gaussian">
+                                <mean>0.0</mean>
+                                <stddev>1.7e-2</stddev>
+                                <bias_mean>0.1</bias_mean>
+                                <bias_stddev>0.001</bias_stddev>
+                            </noise>
+                        </z>
+                    </linear_acceleration>
+                </imu>
+            </sensor>
+        </gazebo>
     </xacro:macro>
     <xacro:base base_link="carcaca" />

File: ros2_ws/src/warehouse_robot/urdf/robot_parts/traction_wheel.xacro (robot description, xacro)
@@ -24,11 +24,13 @@
                 <origin rpy="0 0 0" xyz="0 0 0" />
                 <inertia ixx="0.001" ixy="0.0" ixz="0.0"
-                iyy="0.001" iyz="0.0"
-                izz="0.001" />
+                    iyy="0.001" iyz="0.0"
+                    izz="0.001" />
             </inertial>
             <collision name="${prefix}_collision">
                 <origin rpy="0 0 0" xyz="0 0 0" />
                 <geometry>
-                    <mesh filename="$(find warehouse_robot)/models/laser_robot/wheel/meshes/roda.obj" scale="1 1 1" />
+                    <mesh
+                        filename="$(find warehouse_robot)/models/laser_robot/wheel/meshes/roda.obj"
+                        scale="1 1 1" />
                 </geometry>
             </collision>
@@ -36,10 +38,33 @@
                 <origin rpy="0 0 0" xyz="0 0 0" />
                 <geometry>
-                    <mesh filename="$(find warehouse_robot)/models/laser_robot/wheel/meshes/roda.obj" scale="1 1 1" />
+                    <mesh
+                        filename="$(find warehouse_robot)/models/laser_robot/wheel/meshes/roda.obj"
+                        scale="1 1 1" />
                 </geometry>
             </visual>
         </link>
     </xacro:macro>
-    <xacro:traction_wheel prefix="left_wheel" pos_X="0" pos_Y="0.193" pos_Z="0.0507" pos_r="-1.57" pos_p="0" pos_y="0" axis="1"/>
-    <xacro:traction_wheel prefix="right_wheel" pos_X="0" pos_Y="-0.193" pos_Z="0.0507" pos_r="1.57" pos_p="0" pos_y="0" axis="-1"/>
+    <xacro:traction_wheel prefix="left_wheel" pos_X="0" pos_Y="0.193" pos_Z="0.0507" pos_r="-1.57"
+        pos_p="0" pos_y="0" axis="1" />
+    <xacro:traction_wheel prefix="right_wheel" pos_X="0" pos_Y="-0.193" pos_Z="0.0507" pos_r="1.57"
+        pos_p="0" pos_y="0" axis="-1" />
+    <gazebo>
+        <plugin name='diff_drive' filename='libgazebo_ros_diff_drive.so'>
+            <!-- wheels -->
+            <left_joint>left_wheel_joint</left_joint>
+            <right_joint>right_wheel_joint</right_joint>
+            <!-- kinematics -->
+            <wheel_separation>0.386</wheel_separation>
+            <wheel_diameter>0.0508</wheel_diameter>
+            <!-- limits -->
+            <max_wheel_torque>20</max_wheel_torque>
+            <max_wheel_acceleration>1.0</max_wheel_acceleration>
+            <!-- output -->
+            <publish_odom>true</publish_odom>
+            <publish_odom_tf>false</publish_odom_tf>
+            <publish_wheel_tf>true</publish_wheel_tf>
+            <odometry_frame>odom</odometry_frame>
+            <robot_base_frame>base_link</robot_base_frame>
+        </plugin>
+    </gazebo>
 </robot>

File: ros2_ws/src/warehouse_robot/urdf/ros2_control.xacro (robot description, xacro)
@@ -5,20 +5,4 @@
                 <plugin>gazebo_ros2_control/GazeboSystem</plugin>
             </hardware>
-            <joint name="left_wheel_joint">
-                <command_interface name="velocity">
-                    <param name="min">-10</param>
-                    <param name="max">10</param>
-                </command_interface>
-                <state_interface name="velocity"/>
-                <state_interface name="position"/>
-            </joint>
-            <joint name="right_wheel_joint">
-                <command_interface name="velocity">
-                    <param name="min">-10</param>
-                    <param name="max">10</param>
-                </command_interface>
-                <state_interface name="velocity"/>
-                <state_interface name="position"/>
-            </joint>
             <joint name="joint_piston">
                 <command_interface name="position">
