Commit message: Renenabled xacro urdf sensors

File: ros2_ws/src/warehouse_robot/urdf/robot.urdf.xacro (robot description, xacro)
@@ -10,17 +10,17 @@
   <xacro:include filename="$(find warehouse_robot)/urdf/robot_parts/omni_wheel.xacro" />
   <!--=========================== SENSORS ===========================-->
-  <!-- <xacro:arg name="sensor_imu" default="true" /> -->
+  <xacro:arg name="sensor_imu" default="true" />
   <xacro:arg name="sensor_lidar" default="true" />
-  <!-- <xacro:arg name="sensor_rplidar" default="true" /> -->
+  <xacro:arg name="sensor_rplidar" default="true" />
   <xacro:arg name="sensor_camera" default="true" />
-  <!-- <xacro:if value="$(arg sensor_imu)">
+  <xacro:if value="$(arg sensor_imu)">
     <xacro:include filename="$(find warehouse_robot)/urdf/sensors/imu.xacro" />
-  </xacro:if> -->
+  </xacro:if>
   <xacro:if value="$(arg sensor_lidar)">
     <xacro:include filename="$(find warehouse_robot)/urdf/sensors/lidar.xacro" />
   </xacro:if>
-  <!-- <xacro:if value="$(arg sensor_rplidar)">
+  <xacro:if value="$(arg sensor_rplidar)">
     <xacro:include filename="$(find warehouse_robot)/urdf/sensors/rplidar.xacro" />
-  </xacro:if> -->
+  </xacro:if>
   <xacro:if value="$(arg sensor_camera)">
     <xacro:include filename="$(find warehouse_robot)/urdf/sensors/camera.xacro" />

File: ros2_ws/src/warehouse_robot/urdf/sensors/rplidar.xacro (robot description, xacro)
@@ -39,5 +39,5 @@
     <parent link="base_link" />
     <child link="rplidar" />
-    <origin rpy="0 0 0" xyz="0.14 -0.17 0.27" />
+    <origin rpy="0 0 0" xyz="0.14 -0.17 0.25" />
   </joint>
   <link name="rplidar">

Commit message: Changed to kiva bot

File: ros2_ws/src/warehouse_robot/urdf/robot.urdf.xacro (robot description, xacro)
@@ -11,12 +11,8 @@
   <!--=========================== SENSORS ===========================-->
   <xacro:arg name="sensor_imu" default="true" />
-  <xacro:arg name="sensor_lidar" default="true" />
   <xacro:arg name="sensor_rplidar" default="true" />
   <xacro:arg name="sensor_camera" default="true" />
   <xacro:if value="$(arg sensor_imu)">
     <xacro:include filename="$(find warehouse_robot)/urdf/sensors/imu.xacro" />
-  </xacro:if>
-  <xacro:if value="$(arg sensor_lidar)">
-    <xacro:include filename="$(find warehouse_robot)/urdf/sensors/lidar.xacro" />
   </xacro:if>
   <xacro:if value="$(arg sensor_rplidar)">

File: ros2_ws/src/warehouse_robot/urdf/robot_parts/carcaca.xacro (robot description, xacro)
@@ -10,4 +10,18 @@
             <fdir1 value="0 0 0" />
         </gazebo>
+        <joint name="base_footprint_joint" type="fixed">
+            <parent link="base_link"/>
+            <child link="base_footprint"/>
+            <origin xyz="0 0 0" rpy="0 0 0"/>
+        </joint>
+        <joint name="chassis_joint" type="fixed">
+            <parent link="base_link"/>
+            <child link="${base_link}"/>
+            <origin xyz="0 0 0" rpy="0 0 0"/>
+        </joint>
+        <link name="base_link">
+        </link>
+        <link name="base_footprint">
+        </link>
         <link name="${base_link}">
             <inertial>
@@ -32,4 +46,4 @@
         </link>
     </xacro:macro>
-    <xacro:base base_link="base_link" />
+    <xacro:base base_link="carcaca" />
 </robot>

File: ros2_ws/src/warehouse_robot/urdf/robot_parts/omni_wheel.xacro (robot description, xacro)
@@ -3,5 +3,5 @@
     <xacro:macro name="omni_wheel" params="prefix pos_X pos_Y pos_Z pos_r pos_p pos_y">
         <joint name="joint_${prefix}_wheel" type="fixed">
-            <parent link="base_link" />
+            <parent link="carcaca" />
             <child link="${prefix}_wheel" />
             <origin rpy="${pos_r} ${pos_p} ${pos_y}" xyz="${pos_X} ${pos_Y} ${pos_Z}" />

File: ros2_ws/src/warehouse_robot/urdf/robot_parts/piston.xacro (robot description, xacro)
@@ -2,6 +2,6 @@
 <robot xmlns:xacro="http://www.ros.org/wiki/xacro">
     <xacro:macro name="piston" params="prefix">
-        <joint name="${prefix}_joint" type="prismatic">
-            <parent link="base_link" />
+        <joint name="joint_${prefix}" type="prismatic">
+            <parent link="carcaca" />
             <child link="${prefix}" />
             <dynamics friction="5.0" />

File: ros2_ws/src/warehouse_robot/urdf/robot_parts/traction_wheel.xacro (robot description, xacro)
@@ -3,5 +3,5 @@
     <xacro:macro name="traction_wheel" params="prefix pos_X pos_Y pos_Z pos_r pos_p pos_y">
         <joint name="${prefix}_joint" type="continuous">
-            <parent link="base_link" />
+            <parent link="carcaca" />
             <child link="${prefix}" />
             <origin rpy="${pos_r} ${pos_p} ${pos_y}" xyz="${pos_X} ${pos_Y} ${pos_Z}" />

File: ros2_ws/src/warehouse_robot/urdf/ros2_control.xacro (robot description, xacro)
@@ -1,35 +1,4 @@
 <?xml version="1.0"?>
 <robot xmlns:xacro="http://www.ros.org/wiki/xacro">
-    <xacro:unless value="$(arg sim_mode)">
-        <ros2_control name="RealRobot" type="system">
-            <hardware>
-                <plugin>diffdrive_arduino/DiffDriveArduino</plugin>
-                <param name="left_wheel_name">left_wheel_joint</param>
-                <param name="right_wheel_name">right_wheel_joint</param>
-                <param name="loop_rate">30</param>
-                <param name="device">/dev/ttyUSB0</param>
-                <param name="baud_rate">57600</param>
-                <param name="timeout">1000</param>
-                <param name="enc_counts_per_rev">3436</param>
-            </hardware>
-            <joint name="left_wheel_joint">
-                <command_interface name="velocity">
-                    <param name="min">-10</param>
-                    <param name="max">10</param>
-                </command_interface>
-                <state_interface name="velocity"/>
-                <state_interface name="position"/>
-            </joint>
-            <joint name="right_wheel_joint">
-                <command_interface name="velocity">
-                    <param name="min">-10</param>
-                    <param name="max">10</param>
-                </command_interface>
-                <state_interface name="velocity"/>
-                <state_interface name="position"/>
-            </joint>
-        </ros2_control>
-    </xacro:unless>
-    <xacro:if value="$(arg sim_mode)">
         <ros2_control name="GazeboSystem" type="system">
             <hardware>
@@ -60,5 +29,4 @@
             </joint>
         </ros2_control>
-    </xacro:if>
     <gazebo>
         <plugin name="gazebo_ros2_control" filename="libgazebo_ros2_control.so">

File: ros2_ws/src/warehouse_robot/urdf/sensors/camera.xacro (robot description, xacro)
@@ -40,5 +40,5 @@
     </gazebo>
     <joint name="camera_joint" type="fixed">
-        <parent link="base_link" />
+        <parent link="carcaca" />
         <child link="camera_link" />
         <origin rpy="0 1.57 0" xyz="0 0 0.0367" />

File: ros2_ws/src/warehouse_robot/urdf/sensors/imu.xacro (robot description, xacro)
@@ -4,5 +4,5 @@
         <plugin name="imu_plugin" filename="libgazebo_ros_imu.so">
           <alwaysOn>true</alwaysOn>
-          <bodyName>base_link</bodyName>
+          <bodyName>carcaca</bodyName>
           <topicName>imu</topicName>
           <serviceName>imu_service</serviceName>

File: ros2_ws/src/warehouse_robot/urdf/sensors/lidar.xacro (robot description, xacro)
@@ -40,5 +40,5 @@
   </gazebo>
   <joint name="laser_joint" type="fixed">
-    <parent link="base_link" />
+    <parent link="carcaca" />
     <child link="laser_frame" />
     <origin rpy="0 0 -1.57" xyz="-0.0005 -0.23 0.109" />

File: ros2_ws/src/warehouse_robot/urdf/sensors/rplidar.xacro (robot description, xacro)
@@ -1,45 +1,22 @@
 <?xml version="1.0"?>
 <robot xmlns:xacro="http://www.ros.org/wiki/xacro">
-  <gazebo reference="rplidar">
-    <sensor type="ray" name="laser_sensor">
-      <pose>0 0 0 0 0 0</pose>
-      <visualize>false</visualize>
-      <update_rate>20</update_rate>
-      <ray>
-        <scan>
-          <horizontal>
-            <samples>${14400/20}</samples>
-            <resolution>1</resolution>
-            <min_angle>-3.14159265359</min_angle>
-            <max_angle>3.14159265359</max_angle>
-          </horizontal>
-        </scan>
-        <range>
-          <min>0.15</min>
-          <max>14.0</max>
-          <resolution>0.01</resolution>
-        </range>
-        <noise>
-          <type>gaussian</type>
-          <!-- Noise parameters based on published spec for Hokuyo laser
-                   achieving "+-30mm" accuracy at range < 10m.  A mean of 0.0m and
-                   stddev of 0.01m will put 99.7% of samples within 0.03m of the true
-                   reading. -->
-          <mean>0.0</mean>
-          <stddev>0.01</stddev>
-        </noise>
-      </ray>
-      <plugin name="gazebo_ros_head_hokuyo_controllerrp" filename="libgazebo_ros_ray_sensor.so">
-        <topicName>/my_robot/rplidar/laser/scan</topicName>
-        <frameName>rplidar</frameName>
-      </plugin>
-    </sensor>
-  </gazebo>
   <joint name="joint_rplidar" type="fixed">
-    <parent link="base_link" />
-    <child link="rplidar" />
+    <parent link="carcaca" />
+    <child link="laser_frame" />
     <origin rpy="0 0 0" xyz="0.14 -0.17 0.255" />
   </joint>
-  <link name="rplidar">
+  <link name="laser_frame">
+    <visual>
+      <origin rpy="0 0 1.20" xyz="-0.03 0.02 -0.02" />
+      <geometry>
+        <mesh filename="$(find warehouse_robot)/models/laser_robot/meshes/rplidar.dae" scale="0.7 0.7 0.7" />
+      </geometry>
+    </visual>
+    <collision>
+      <origin rpy="0 0 1.20" xyz="-0.03 0.02 -0.02" />
+      <geometry>
+        <mesh filename="$(find warehouse_robot)/models/laser_robot/meshes/rplidar.dae" scale="0.7 0.7 0.7" />
+      </geometry>
+    </collision>
     <inertial>
       <mass value="0.1" />
@@ -47,16 +24,31 @@
       <inertia ixx="1" ixy="0" ixz="0" iyy="1" iyz="0" izz="1" />
     </inertial>
-    <collision name="rplidar_collision">
-      <origin rpy="0 0 1.20" xyz="-0.03 0.02 -0.02" />
-      <geometry>
-        <mesh filename="$(find warehouse_robot)/models/laser_robot/meshes/rplidar.dae" scale="0.7 0.7 0.7" />
-      </geometry>
-    </collision>
-    <visual name="rplidar_visual">
-      <origin rpy="0 0 1.20" xyz="-0.03 0.02 -0.02" />
-      <geometry>
-        <mesh filename="$(find warehouse_robot)/models/laser_robot/meshes/rplidar.dae" scale="0.7 0.7 0.7" />
-      </geometry>
-    </visual>
-  </link>
+</link>
+<gazebo reference="laser_frame">
+    <sensor name="laser" type="ray">
+        <pose> 0 0 0 0 0 0 </pose>
+        <visualize>true</visualize>
+        <update_rate>10</update_rate>
+        <ray>
+            <scan>
+                <horizontal>
+                    <samples>360</samples>
+                    <min_angle>-3.14</min_angle>
+                    <max_angle>3.14</max_angle>
+                </horizontal>
+            </scan>
+            <range>
+                <min>0.3</min>
+                <max>12</max>
+            </range>
+        </ray>
+        <plugin name="laser_controller" filename="libgazebo_ros_ray_sensor.so">
+            <ros>
+                <argument>~/out:=scan</argument>
+            </ros>
+            <output_type>sensor_msgs/LaserScan</output_type>
+            <frame_name>laser_frame</frame_name>
+        </plugin>
+    </sensor>
+</gazebo>
 </robot>

Commit message: working version of kiva bot

File: ros2_ws/src/warehouse_robot/urdf/robot.urdf.xacro (robot description, xacro)
@@ -6,19 +6,19 @@
   <xacro:include filename="$(find warehouse_robot)/urdf/robot_parts/carcaca.xacro" />
   <xacro:include filename="$(find warehouse_robot)/urdf/robot_parts/traction_wheel.xacro" />
-  <xacro:include filename="$(find warehouse_robot)/urdf/robot_parts/tray.xacro" />
-  <xacro:include filename="$(find warehouse_robot)/urdf/robot_parts/piston.xacro" />
+  <!-- <xacro:include filename="$(find warehouse_robot)/urdf/robot_parts/tray.xacro" /> -->
+  <!-- <xacro:include filename="$(find warehouse_robot)/urdf/robot_parts/piston.xacro" /> -->
   <xacro:include filename="$(find warehouse_robot)/urdf/robot_parts/omni_wheel.xacro" />
   <!--=========================== SENSORS ===========================-->
-  <xacro:arg name="sensor_imu" default="true" />
+  <!-- <xacro:arg name="sensor_imu" default="true" /> -->
   <xacro:arg name="sensor_rplidar" default="true" />
-  <xacro:arg name="sensor_camera" default="true" />
-  <xacro:if value="$(arg sensor_imu)">
+  <!-- <xacro:arg name="sensor_camera" default="true" /> -->
+  <!-- <xacro:if value="$(arg sensor_imu)">
     <xacro:include filename="$(find warehouse_robot)/urdf/sensors/imu.xacro" />
-  </xacro:if>
+  </xacro:if> -->
   <xacro:if value="$(arg sensor_rplidar)">
     <xacro:include filename="$(find warehouse_robot)/urdf/sensors/rplidar.xacro" />
   </xacro:if>
-  <xacro:if value="$(arg sensor_camera)">
+  <!-- <xacro:if value="$(arg sensor_camera)">
     <xacro:include filename="$(find warehouse_robot)/urdf/sensors/camera.xacro" />
-  </xacro:if>
+  </xacro:if> -->
 </robot>

File: ros2_ws/src/warehouse_robot/urdf/robot_parts/carcaca.xacro (robot description, xacro)
@@ -3,5 +3,5 @@
     <xacro:macro name="base" params="base_link">
         <gazebo reference="${base_link}">
-            <selfCollide>true</selfCollide>
+            <selfCollide>false</selfCollide>
             <mu1 value="0.3" />
             <mu2 value="0.3" />
@@ -27,5 +27,5 @@
             <inertial>
                 <mass value="2.4" />
-                <origin rpy="0  0  3.14" xyz="0  0  0.0118" />
+                <origin rpy="0  0  0" xyz="0  0  0.0118" />
                 <inertia ixx="0.019995" ixy="0.0" ixz="0.0"
                 iyy="0.019995" iyz="0.0"
@@ -33,5 +33,5 @@
             </inertial>
             <collision name="${base_link}_collision">
-                <origin rpy="0  0  3.14" xyz="0  0  0.0118" />
+                <origin rpy="0  0  0" xyz="0  0  0.0118" />
                 <geometry>
                     <mesh filename="$(find warehouse_robot)/models/laser_robot/meshes/carcaca.dae" scale="1 1 1" />
@@ -39,5 +39,5 @@
             </collision>
             <visual name="${base_link}_visual">
-                <origin rpy="0  0  3.14" xyz="0  0  0.0118" />
+                <origin rpy="0  0  0" xyz="0  0  0.0118" />
                 <geometry>
                     <mesh filename="$(find warehouse_robot)/models/laser_robot/meshes/carcaca.dae" scale="1 1 1" />

File: ros2_ws/src/warehouse_robot/urdf/robot_parts/omni_wheel.xacro (robot description, xacro)
@@ -35,7 +35,7 @@
         </link>
     </xacro:macro>
-    <xacro:omni_wheel prefix="left_front" pos_X="-0.214" pos_Y="-0.176" pos_Z="0.0508" pos_r="0" pos_p="1.57" pos_y="0" />
-    <xacro:omni_wheel prefix="left_rear" pos_X="-0.214" pos_Y="0.176" pos_Z="0.0508" pos_r="0" pos_p="1.57" pos_y="0" />
-    <xacro:omni_wheel prefix="right_front" pos_X="0.193" pos_Y="-0.176" pos_Z="0.0508" pos_r="0" pos_p="1.57" pos_y="0" />
-    <xacro:omni_wheel prefix="right_rear" pos_X="0.193" pos_Y="0.176" pos_Z="0.0508" pos_r="0" pos_p="1.57" pos_y="0" />
+    <xacro:omni_wheel prefix="left_front" pos_X="0.193" pos_Y="-0.176" pos_Z="0.0508" pos_r="-1.57" pos_p="0" pos_y="0" />
+    <xacro:omni_wheel prefix="left_rear" pos_X="0.193" pos_Y="0.176" pos_Z="0.0508" pos_r="-1.57" pos_p="0" pos_y="0" />
+    <xacro:omni_wheel prefix="right_front" pos_X="-0.214" pos_Y="-0.176" pos_Z="0.0508" pos_r="1.57" pos_p="0" pos_y="0" />
+    <xacro:omni_wheel prefix="right_rear" pos_X="-0.214" pos_Y="0.176" pos_Z="0.0508" pos_r="1.57" pos_p="0" pos_y="0" />
 </robot>

File: ros2_ws/src/warehouse_robot/urdf/robot_parts/traction_wheel.xacro (robot description, xacro)
@@ -1,11 +1,11 @@
 <?xml version="1.0"?>
 <robot xmlns:xacro="http://www.ros.org/wiki/xacro">
-    <xacro:macro name="traction_wheel" params="prefix pos_X pos_Y pos_Z pos_r pos_p pos_y">
+    <xacro:macro name="traction_wheel" params="prefix pos_X pos_Y pos_Z pos_r pos_p pos_y axis">
         <joint name="${prefix}_joint" type="continuous">
             <parent link="carcaca" />
             <child link="${prefix}" />
             <origin rpy="${pos_r} ${pos_p} ${pos_y}" xyz="${pos_X} ${pos_Y} ${pos_Z}" />
-            <axis xyz="0 0 1" />
-            <limit effort="-1.0" lower="-1e+16" upper="1e+16" velocity="-1.0" />
+            <axis xyz="0 0 ${axis}" />
+            <!-- <limit effort="-1.0" lower="-1e+16" upper="1e+16" velocity="-1.0" /> -->
         </joint>
         <gazebo reference="${prefix}">
@@ -41,5 +41,5 @@
         </link>
     </xacro:macro>
-    <xacro:traction_wheel prefix="left_wheel" pos_X="-0.214" pos_Y="0" pos_Z="0.0507" pos_r="0" pos_p="1.57" pos_y="0" />
-    <xacro:traction_wheel prefix="right_wheel" pos_X="0.193" pos_Y="0" pos_Z="0.0507" pos_r="0" pos_p="1.57" pos_y="0" />
+    <xacro:traction_wheel prefix="left_wheel" pos_X="0" pos_Y="0.193" pos_Z="0.0507" pos_r="-1.57" pos_p="0" pos_y="0" axis="1"/>
+    <xacro:traction_wheel prefix="right_wheel" pos_X="0" pos_Y="-0.214" pos_Z="0.0507" pos_r="1.57" pos_p="0" pos_y="0" axis="-1"/>
 </robot>

File: ros2_ws/src/warehouse_robot/urdf/sensors/rplidar.xacro (robot description, xacro)
@@ -1,5 +1,5 @@
 <?xml version="1.0"?>
 <robot xmlns:xacro="http://www.ros.org/wiki/xacro">
-  <joint name="joint_rplidar" type="fixed">
+  <joint name="laser_joint" type="fixed">
     <parent link="carcaca" />
     <child link="laser_frame" />

Commit message: Tuned amcl

File: ros2_ws/src/warehouse_robot/urdf/robot.urdf.xacro (robot description, xacro)
@@ -6,6 +6,6 @@
   <xacro:include filename="$(find warehouse_robot)/urdf/robot_parts/carcaca.xacro" />
   <xacro:include filename="$(find warehouse_robot)/urdf/robot_parts/traction_wheel.xacro" />
-  <xacro:include filename="$(find warehouse_robot)/urdf/robot_parts/tray.xacro" />
-  <xacro:include filename="$(find warehouse_robot)/urdf/robot_parts/piston.xacro" />
+  <!-- <xacro:include filename="$(find warehouse_robot)/urdf/robot_parts/tray.xacro" /> -->
+  <!-- <xacro:include filename="$(find warehouse_robot)/urdf/robot_parts/piston.xacro" /> -->
   <xacro:include filename="$(find warehouse_robot)/urdf/robot_parts/omni_wheel.xacro" />
   <!--=========================== SENSORS ===========================-->

File: ros2_ws/src/warehouse_robot/urdf/robot_parts/piston.xacro (robot description, xacro)
@@ -3,5 +3,5 @@
     <xacro:macro name="piston" params="prefix">
         <joint name="joint_${prefix}" type="prismatic">
-            <parent link="carcaca" />
+            <parent link="base_link" />
             <child link="${prefix}" />
             <dynamics friction="5.0" />

File: ros2_ws/src/warehouse_robot/urdf/ros2_control.xacro (robot description, xacro)
@@ -21,5 +21,5 @@
                 <state_interface name="position"/>
             </joint>
-            <joint name="joint_piston">
+            <!-- <joint name="joint_piston">
                 <command_interface name="position">
                     <param name="min">-10</param>
@@ -27,5 +27,5 @@
                 </command_interface>
                 <state_interface name="position"/>
-            </joint>
+            </joint> -->
         </ros2_control>
     <gazebo>
@@ -35,5 +35,5 @@
         </plugin>
     </gazebo>
-    <transmission name="tran1">
+    <!-- <transmission name="tran1">
         <type>transmission_interface/SimpleTransmission</type>
         <joint name="joint_piston">
@@ -44,4 +44,4 @@
           <mechanicalReduction>1</mechanicalReduction>
         </actuator>
-    </transmission>
+    </transmission> -->
 </robot>

File: ros2_ws/src/warehouse_robot/urdf/sensors/camera.xacro (robot description, xacro)
@@ -39,5 +39,5 @@
     </gazebo>
     <joint name="camera_joint" type="fixed">
-        <parent link="carcaca" />
+        <parent link="base_link" />
         <child link="camera_link" />
         <origin rpy="0 1.57 0" xyz="0 0 0.0367" />

File: ros2_ws/src/warehouse_robot/urdf/sensors/rplidar.xacro (robot description, xacro)
@@ -2,5 +2,5 @@
 <robot xmlns:xacro="http://www.ros.org/wiki/xacro">
   <joint name="laser_joint" type="fixed">
-    <parent link="carcaca" />
+    <parent link="base_link" />
     <child link="laser_frame" />
     <origin rpy="0 0 0" xyz="0.14 -0.17 0.255" />
@@ -14,5 +14,5 @@
     </visual>
     <collision>
-      <origin rpy="0 0 1.20" xyz="-0.03 0.02 -0.02" />
+      <origin rpy="0 0 1.20" xyz="-0.03 0.02 -0.1" />
       <geometry>
         <mesh filename="$(find warehouse_robot)/models/laser_robot/meshes/rplidar.dae" scale="0.7 0.7 0.7" />
@@ -26,4 +26,5 @@
 </link>
 <gazebo reference="laser_frame">
+  <selfCollision>false</selfCollision>
     <sensor name="laser" type="ray">
         <pose> 0 0 0 0 0 0 </pose>

Commit message: enabled the piston

File: ros2_ws/src/warehouse_robot/urdf/robot.urdf.xacro (robot description, xacro)
@@ -6,6 +6,6 @@
   <xacro:include filename="$(find warehouse_robot)/urdf/robot_parts/carcaca.xacro" />
   <xacro:include filename="$(find warehouse_robot)/urdf/robot_parts/traction_wheel.xacro" />
-  <!-- <xacro:include filename="$(find warehouse_robot)/urdf/robot_parts/tray.xacro" /> -->
-  <!-- <xacro:include filename="$(find warehouse_robot)/urdf/robot_parts/piston.xacro" /> -->
+  <xacro:include filename="$(find warehouse_robot)/urdf/robot_parts/tray.xacro" />
+  <xacro:include filename="$(find warehouse_robot)/urdf/robot_parts/piston.xacro" />
   <xacro:include filename="$(find warehouse_robot)/urdf/robot_parts/omni_wheel.xacro" />
   <!--=========================== SENSORS ===========================-->

File: ros2_ws/src/warehouse_robot/urdf/ros2_control.xacro (robot description, xacro)
@@ -21,5 +21,5 @@
                 <state_interface name="position"/>
             </joint>
-            <!-- <joint name="joint_piston">
+            <joint name="joint_piston">
                 <command_interface name="position">
                     <param name="min">-10</param>
@@ -27,5 +27,5 @@
                 </command_interface>
                 <state_interface name="position"/>
-            </joint> -->
+            </joint>
         </ros2_control>
     <gazebo>
@@ -35,5 +35,5 @@
         </plugin>
     </gazebo>
-    <!-- <transmission name="tran1">
+    <transmission name="tran1">
         <type>transmission_interface/SimpleTransmission</type>
         <joint name="joint_piston">
@@ -44,4 +44,4 @@
           <mechanicalReduction>1</mechanicalReduction>
         </actuator>
-    </transmission> -->
+    </transmission>
 </robot>
