Commit message: fixed piston control

File: ros2_ws/src/warehouse_robot/urdf/robot.urdf.xacro (robot description, xacro)
@@ -2,5 +2,5 @@
 <robot name="my_robot" xmlns:xacro="http://www.ros.org/wiki/xacro">
   <!--=========================== PLUGINS ===========================-->
-  <!-- <xacro:include filename="$(find warehouse_robot)/urdf/ros2_control.xacro" /> -->
+  <xacro:include filename="$(find warehouse_robot)/urdf/ros2_control.xacro" />
   <!--=========================== ROBOT PARTS ===========================-->
   <xacro:include filename="$(find warehouse_robot)/urdf/robot_parts/carcaca.xacro" />
@@ -12,3 +12,7 @@
     <xacro:include filename="$(find warehouse_robot)/urdf/sensors/rplidar.xacro" />
     <xacro:include filename="$(find warehouse_robot)/urdf/sensors/camera.xacro" />
+<!-- <gazebo>
+    <plugin name="gazebo_ros_control" filename="libgazebo_ros_control.so">
+    </plugin>
+  </gazebo> -->
 </robot>

File: ros2_ws/src/warehouse_robot/urdf/robot_parts/piston.xacro (robot description, xacro)
@@ -27,5 +27,6 @@
                 <origin rpy="0  0  0" xyz="0 0 0" />
                 <geometry>
-                    <mesh filename="$(find warehouse_robot)/models/laser_robot/meshes/piston.dae" scale="1 1 1" />
+                    <mesh filename="$(find warehouse_robot)/models/laser_robot/meshes/piston.dae"
+                        scale="1 1 1" />
                 </geometry>
             </collision>
@@ -33,8 +34,24 @@
                 <origin rpy="0  0  0" xyz="0 0 0" />
                 <geometry>
-                    <mesh filename="$(find warehouse_robot)/models/laser_robot/meshes/piston.dae" scale="1 1 1" />
+                    <mesh filename="$(find warehouse_robot)/models/laser_robot/meshes/piston.dae"
+                        scale="1 1 1" />
                 </geometry>
             </visual>
         </link>
+        <!-- <transmission name="tran1">
+            <type>transmission_interface/SimpleTransmission</type>
+            <joint name="joint_piston">
+                <hardwareInterface>hardware_interface/EffortJointInterface</hardwareInterface>
+            </joint>
+            <actuator name="motor1">
+                <hardwareInterface>hardware_interface/EffortJointInterface</hardwareInterface>
+                <mechanicalReduction>1</mechanicalReduction>
+            </actuator>
+        </transmission>
+        <gazebo>
+            <plugin name="joint_state_publisher" filename="libgazebo_ros_joint_state_publisher.so">
+                <jointName>joint_piston, joint_tray</jointName>
+            </plugin>
+        </gazebo> -->
     </xacro:macro>
     <xacro:piston prefix="piston" />

File: ros2_ws/src/warehouse_robot/urdf/robot_parts/traction_wheel.xacro (robot description, xacro)
@@ -58,6 +58,6 @@
             <wheel_diameter>0.0508</wheel_diameter>
             <!-- limits -->
-            <max_wheel_torque>20</max_wheel_torque>
-            <max_wheel_acceleration>1.0</max_wheel_acceleration>
+            <max_wheel_torque>3</max_wheel_torque>
+            <max_wheel_acceleration>0</max_wheel_acceleration>
             <!-- output -->
             <publish_odom>true</publish_odom>

File: ros2_ws/src/warehouse_robot/urdf/ros2_control.xacro (robot description, xacro)
@@ -19,13 +19,3 @@
         </plugin>
     </gazebo>
-    <transmission name="tran1">
-        <type>transmission_interface/SimpleTransmission</type>
-        <joint name="joint_piston">
-          <hardwareInterface>hardware_interface/EffortJointInterface</hardwareInterface>
-        </joint>
-        <actuator name="motor1">
-          <hardwareInterface>hardware_interface/EffortJointInterface</hardwareInterface>
-          <mechanicalReduction>1</mechanicalReduction>
-        </actuator>
-    </transmission>
 </robot>
