Commit message: Started simplifying launch scripts to just spawn robot in gazebo

File: ros2_ws/src/warehouse_robot/urdf/robot_1.urdf.xacro (robot description, xacro)
@@ -2,13 +2,13 @@
 <robot name="my_robot_1" xmlns:xacro="http://www.ros.org/wiki/xacro">
   <!--=========================== PLUGINS ===========================-->
-  <xacro:include filename="$(find warehouse_robot)/urdf/ros2_control.xacro" ns="robot_1" />
+  <!-- <xacro:include filename="$(find warehouse_robot)/urdf/ros2_control.xacro" ns="robot_1" /> -->
   <!--=========================== ROBOT PARTS ===========================-->
-  <xacro:include filename="$(find warehouse_robot)/urdf/robot_parts/carcaca.xacro" ns="robot_1"/>
-  <xacro:include filename="$(find warehouse_robot)/urdf/robot_parts/traction_wheel.xacro" ns="robot_1"/>
-  <xacro:include filename="$(find warehouse_robot)/urdf/robot_parts/tray.xacro" ns="robot_1"/>
-  <xacro:include filename="$(find warehouse_robot)/urdf/robot_parts/piston.xacro" ns="robot_1"/>
-  <xacro:include filename="$(find warehouse_robot)/urdf/robot_parts/omni_wheel.xacro" ns="robot_1"/>
+  <xacro:include filename="$(find warehouse_robot)/urdf/robot_parts/carcaca.xacro"/>
+  <xacro:include filename="$(find warehouse_robot)/urdf/robot_parts/traction_wheel.xacro"/>
+  <xacro:include filename="$(find warehouse_robot)/urdf/robot_parts/tray.xacro"/>
+  <xacro:include filename="$(find warehouse_robot)/urdf/robot_parts/piston.xacro"/>
+  <xacro:include filename="$(find warehouse_robot)/urdf/robot_parts/omni_wheel.xacro"/>
   <!--=========================== SENSORS ===========================-->
-    <xacro:include filename="$(find warehouse_robot)/urdf/sensors/rplidar.xacro" ns="robot_1"/>
-    <xacro:include filename="$(find warehouse_robot)/urdf/sensors/camera.xacro" ns="robot_1"/>
+    <xacro:include filename="$(find warehouse_robot)/urdf/sensors/rplidar.xacro"/>
+    <xacro:include filename="$(find warehouse_robot)/urdf/sensors/camera.xacro"/>
 </robot>

File: ros2_ws/src/warehouse_robot/urdf/robot_2.urdf.xacro (robot description, xacro)
@@ -2,13 +2,13 @@
 <robot name="my_robot_2" xmlns:xacro="http://www.ros.org/wiki/xacro">
   <!--=========================== PLUGINS ===========================-->
-  <xacro:include filename="$(find warehouse_robot)/urdf/ros2_control.xacro" ns="robot_2"/>
+  <!-- <xacro:include filename="$(find warehouse_robot)/urdf/ros2_control.xacro" ns="robot_2"/> -->
   <!--=========================== ROBOT PARTS ===========================-->
-  <xacro:include filename="$(find warehouse_robot)/urdf/robot_parts/carcaca.xacro" ns="robot_2"/>
-  <xacro:include filename="$(find warehouse_robot)/urdf/robot_parts/traction_wheel.xacro" ns="robot_2"/>
-  <xacro:include filename="$(find warehouse_robot)/urdf/robot_parts/tray.xacro" ns="robot_2" />
-  <xacro:include filename="$(find warehouse_robot)/urdf/robot_parts/piston.xacro" ns="robot_2"/>
-  <xacro:include filename="$(find warehouse_robot)/urdf/robot_parts/omni_wheel.xacro" ns="robot_2"/>
+  <xacro:include filename="$(find warehouse_robot)/urdf/robot_parts/carcaca.xacro"/>
+  <xacro:include filename="$(find warehouse_robot)/urdf/robot_parts/traction_wheel.xacro"/>
+  <xacro:include filename="$(find warehouse_robot)/urdf/robot_parts/tray.xacro"/>
+  <xacro:include filename="$(find warehouse_robot)/urdf/robot_parts/piston.xacro"/>
+  <xacro:include filename="$(find warehouse_robot)/urdf/robot_parts/omni_wheel.xacro"/>
   <!--=========================== SENSORS ===========================-->
-    <xacro:include filename="$(find warehouse_robot)/urdf/sensors/rplidar.xacro" ns="robot_2"/>
-    <xacro:include filename="$(find warehouse_robot)/urdf/sensors/camera.xacro" ns="robot_2"/>
+    <xacro:include filename="$(find warehouse_robot)/urdf/sensors/rplidar.xacro"/>
+    <xacro:include filename="$(find warehouse_robot)/urdf/sensors/camera.xacro"/>
 </robot>

File: ros2_ws/src/warehouse_robot/urdf/robot_3.urdf.xacro (robot description, xacro)
@@ -2,5 +2,5 @@
 <robot name="my_robot_3" xmlns:xacro="http://www.ros.org/wiki/xacro">
   <!--=========================== PLUGINS ===========================-->
-  <xacro:include filename="$(find warehouse_robot)/urdf/ros2_control.xacro" />
+  <!-- <xacro:include filename="$(find warehouse_robot)/urdf/ros2_control.xacro" /> -->
   <!--=========================== ROBOT PARTS ===========================-->
   <xacro:include filename="$(find warehouse_robot)/urdf/robot_parts/carcaca.xacro" />

File: ros2_ws/src/warehouse_robot/urdf/robot_4.urdf.xacro (robot description, xacro)
@@ -2,5 +2,5 @@
 <robot name="my_robot_4" xmlns:xacro="http://www.ros.org/wiki/xacro">
   <!--=========================== PLUGINS ===========================-->
-  <xacro:include filename="$(find warehouse_robot)/urdf/ros2_control.xacro" />
+  <!-- <xacro:include filename="$(find warehouse_robot)/urdf/ros2_control.xacro" /> -->
   <!--=========================== ROBOT PARTS ===========================-->
   <xacro:include filename="$(find warehouse_robot)/urdf/robot_parts/carcaca.xacro" />

File: ros2_ws/src/warehouse_robot/urdf/robot_5.urdf.xacro (robot description, xacro)
@@ -2,5 +2,5 @@
 <robot name="my_robot_5" xmlns:xacro="http://www.ros.org/wiki/xacro">
   <!--=========================== PLUGINS ===========================-->
-  <xacro:include filename="$(find warehouse_robot)/urdf/ros2_control.xacro" />
+  <!-- <xacro:include filename="$(find warehouse_robot)/urdf/ros2_control.xacro" /> -->
   <!--=========================== ROBOT PARTS ===========================-->
   <xacro:include filename="$(find warehouse_robot)/urdf/robot_parts/carcaca.xacro" />

File: ros2_ws/src/warehouse_robot/urdf/robot_parts/omni_wheel.xacro (robot description, xacro)
@@ -1,5 +1,5 @@
 <?xml version="1.0"?>
 <robot xmlns:xacro="http://www.ros.org/wiki/xacro">
-    <xacro:macro name="omni_wheel" params="namespace prefix pos_X pos_Y pos_Z pos_r pos_p pos_y">
+    <xacro:macro name="omni_wheel" params="prefix pos_X pos_Y pos_Z pos_r pos_p pos_y">
         <joint name="joint_${prefix}_wheel" type="fixed">
             <parent link="base_link" />

File: ros2_ws/src/warehouse_robot/urdf/robot_parts/piston.xacro (robot description, xacro)
@@ -1,5 +1,5 @@
 <?xml version="1.0"?>
 <robot xmlns:xacro="http://www.ros.org/wiki/xacro">
-    <xacro:macro name="piston" params="namespace prefix">
+    <xacro:macro name="piston" params="prefix">
         <joint name="joint_${prefix}" type="prismatic">
             <parent link="carcaca" />

File: ros2_ws/src/warehouse_robot/urdf/robot_parts/traction_wheel.xacro (robot description, xacro)
@@ -1,5 +1,5 @@
 <?xml version="1.0"?>
 <robot xmlns:xacro="http://www.ros.org/wiki/xacro">
-    <xacro:macro name="traction_wheel" params="namespace prefix pos_X pos_Y pos_Z pos_r pos_p pos_y axis">
+    <xacro:macro name="traction_wheel" params="prefix pos_X pos_Y pos_Z pos_r pos_p pos_y axis">
         <joint name="${prefix}_joint" type="continuous">
             <parent link="base_link" />

File: ros2_ws/src/warehouse_robot/urdf/robot_parts/tray.xacro (robot description, xacro)
@@ -1,5 +1,5 @@
 <?xml version="1.0"?>
 <robot xmlns:xacro="http://www.ros.org/wiki/xacro">
-    <xacro:macro name="tray" params="namespace prefix">
+    <xacro:macro name="tray" params="prefix">
         <joint name="joint_${prefix}" type="continuous">
             <parent link="piston" />
