Commit message: Added piston control to warehouse robot

File: ros2_ws/src/warehouse_robot/urdf/robot_parts/piston.xacro (robot description, xacro)
@@ -2,5 +2,5 @@
 <robot xmlns:xacro="http://www.ros.org/wiki/xacro">
     <xacro:macro name="piston" params="prefix">
-        <joint name="joint_${prefix}" type="prismatic">
+        <joint name="${prefix}_joint" type="prismatic">
             <parent link="base_link" />
             <child link="${prefix}" />

File: ros2_ws/src/warehouse_robot/urdf/ros2_control.xacro (robot description, xacro)
@@ -52,4 +52,11 @@
                 <state_interface name="position"/>
             </joint>
+            <joint name="piston_joint">
+                <command_interface name="position">
+                    <param name="min">-10</param>
+                    <param name="max">10</param>
+                </command_interface>
+                <state_interface name="position"/>
+            </joint>
         </ros2_control>
     </xacro:if>

Commit message: Attempted to add transmission control

File: ros2_ws/src/warehouse_robot/urdf/robot_parts/piston.xacro (robot description, xacro)
@@ -5,5 +5,5 @@
             <parent link="base_link" />
             <child link="${prefix}" />
-            <!-- <dynamics friction="5.0" /> -->
+            <dynamics friction="5.0" />
             <origin rpy="0 0 0" xyz="0 0 0.1318" />
             <axis xyz="0 0 1" />

File: ros2_ws/src/warehouse_robot/urdf/ros2_control.xacro (robot description, xacro)
@@ -67,3 +67,13 @@
         </plugin>
     </gazebo>
+    <transmission name="tran1">
+        <type>transmission_interface/SimpleTransmission</type>
+        <joint name="piston_joint">
+          <hardwareInterface>hardware_interface/EffortJointInterface</hardwareInterface>
+        </joint>
+        <actuator name="motor1">
+          <hardwareInterface>hardware_interface/EffortJointInterface</hardwareInterface>
+          <mechanicalReduction>1</mechanicalReduction>
+        </actuator>
+    </transmission>
 </robot>

Commit message: Switch piston controller to position_controllers/JointGroupPositionController and did some tuning

File: ros2_ws/src/warehouse_robot/urdf/robot_parts/piston.xacro (robot description, xacro)
@@ -8,5 +8,5 @@
             <origin rpy="0 0 0" xyz="0 0 0.1318" />
             <axis xyz="0 0 1" />
-            <limit effort="0" lower="0" upper="0.04" velocity="0" />
+            <limit effort="0" lower="0" upper="0.05" velocity="0" />
         </joint>
         <gazebo reference="${prefix}">
@@ -15,5 +15,5 @@
             <mu2 value="0.1" />
             <kp value="10000000.0" />
-            <kd value="10000" />
+            <kd value="1000000" />
             <fdir1 value="0 0 0" />
         </gazebo>

File: ros2_ws/src/warehouse_robot/urdf/robot_parts/tray.xacro (robot description, xacro)
@@ -5,5 +5,5 @@
             <parent link="piston" />
             <child link="${prefix}" />
-            <!-- <dynamics friction="5.0" /> -->
+            <dynamics friction="5.0" />
             <origin rpy="0 0 0" xyz="0 0 0" />
             <axis xyz="0 0 1" />

File: ros2_ws/src/warehouse_robot/urdf/ros2_control.xacro (robot description, xacro)
@@ -27,4 +27,5 @@
                 </command_interface>
                 <state_interface name="position"/>
+                <state_interface name="velocity"/>
             </joint>
         </ros2_control>

Commit message: A lot of changes that didn't work, but switched piston to velocity controller

File: ros2_ws/src/warehouse_robot/urdf/robot_parts/piston.xacro (robot description, xacro)
@@ -5,8 +5,8 @@
             <parent link="base_link" />
             <child link="${prefix}" />
-            <dynamics friction="5.0" />
+            <!-- <dynamics friction="5.0" /> -->
             <origin rpy="0 0 0" xyz="0 0 0.1318" />
             <axis xyz="0 0 1" />
-            <limit effort="0" lower="0" upper="0.05" velocity="0" />
+            <limit effort="1" lower="0" upper="0.05" velocity=".00005" />
         </joint>
         <gazebo reference="${prefix}">
@@ -14,6 +14,6 @@
             <mu1 value="0.1" />
             <mu2 value="0.1" />
-            <kp value="10000000.0" />
-            <kd value="1000000" />
+            <kp value=".00001" />
+            <kd value="10000000" />
             <fdir1 value="0 0 0" />
         </gazebo>

File: ros2_ws/src/warehouse_robot/urdf/ros2_control.xacro (robot description, xacro)
@@ -26,4 +26,8 @@
                     <param name="max">10</param>
                 </command_interface>
+                <command_interface name="velocity">
+                    <param name="min">-.1</param>
+                    <param name="max">.001</param>
+                </command_interface>
                 <state_interface name="position"/>
                 <state_interface name="velocity"/>
