Commit message: fixed the orientation of the camera

File: ros2_ws/src/warehouse_robot/urdf/robot_parts/carcaca.xacro (robot description, xacro)
@@ -27,5 +27,5 @@
             <inertial>
                 <mass value="2.4" />
-                <origin rpy="0  0  0" xyz="0  0  0.0118" />
+                <origin rpy="0  0  0" xyz="0.017  0  0.0118" />
                 <inertia ixx="0.019995" ixy="0.0" ixz="0.0"
                 iyy="0.019995" iyz="0.0"

File: ros2_ws/src/warehouse_robot/urdf/sensors/camera.xacro (robot description, xacro)
@@ -5,5 +5,5 @@
             <update_rate>30.0</update_rate>
             <visualize>true</visualize>
-            <camera name="camera">
+            <camera>
                 <horizontal_fov>1.3962634</horizontal_fov>
                 <image>
@@ -16,9 +16,9 @@
                     <far>300</far>
                 </clip>
-                <noise>
+                <!-- <noise>
                     <type>gaussian</type>
                     <mean>0.0</mean>
                     <stddev>0.007</stddev>
-                </noise>
+                </noise> -->
             </camera>
             <plugin name="camera_controller" filename="libgazebo_ros_camera.so">
@@ -40,25 +40,14 @@
     <joint name="camera_joint" type="fixed">
         <parent link="carcaca" />
-        <child link="camera_link_optical" />
+        <child link="camera_link" />
         <origin rpy="0 1.57 0" xyz="0 0 0.0367" />
     </joint>
-    <link name="camera_link_optical">
-        <inertial>
-            <mass value="0.1" />
-            <origin rpy="0 0 0" xyz="0 0 0" />
-            <inertia ixx="1" ixy="0" ixz="0" iyy="1" iyz="0" izz="1" />
-        </inertial>
-        <collision>
-            <origin rpy="0 0 0" xyz="0 0 0" />
-            <geometry>
-                <mesh filename="$(find warehouse_robot)/models/laser_robot/camera/meshes/camera.obj" scale="0.5 0.5 0.5" />
-            </geometry>
-        </collision>
-        <visual>
-            <origin rpy="0 0 1.57" xyz="0 0 0" />
-            <geometry>
-                <mesh filename="$(find warehouse_robot)/models/laser_robot/camera/meshes/camera.obj" scale="0.5 0.5 0.5" />
-            </geometry>
-        </visual>
+    <joint name="camera_optical_joint" type="fixed">
+        <parent link="camera_link" />
+        <child link="camera_link_optical" />
+        <origin rpy="-1.57 0 -1.57" xyz="0 0 0" />
+    </joint>
+    <link name="camera_link">
     </link>
+    <link name="camera_link_optical"></link>
 </robot>

Commit message: enabled collision

File: ros2_ws/src/warehouse_robot/urdf/robot_parts/carcaca.xacro (robot description, xacro)
@@ -3,5 +3,5 @@
     <xacro:macro name="base" params="base_link">
         <gazebo reference="${base_link}">
-            <selfCollide>false</selfCollide>
+            <selfCollide>true</selfCollide>
             <mu1 value="0.3" />
             <mu2 value="0.3" />
@@ -18,5 +18,5 @@
             <parent link="base_link"/>
             <child link="${base_link}"/>
-            <origin xyz="0 0 0" rpy="0 0 0"/>
+            <origin xyz="0 0 0" rpy="0 0 -1.57"/>
         </joint>
         <link name="base_link">
@@ -27,5 +27,5 @@
             <inertial>
                 <mass value="2.4" />
-                <origin rpy="0  0  0" xyz="0.017  0  0.0118" />
+                <origin rpy="0  0  0" xyz="0  0  0.0118" />
                 <inertia ixx="0.019995" ixy="0.0" ixz="0.0"
                 iyy="0.019995" iyz="0.0"

File: ros2_ws/src/warehouse_robot/urdf/robot_parts/omni_wheel.xacro (robot description, xacro)
@@ -3,10 +3,10 @@
     <xacro:macro name="omni_wheel" params="prefix pos_X pos_Y pos_Z pos_r pos_p pos_y">
         <joint name="joint_${prefix}_wheel" type="fixed">
-            <parent link="carcaca" />
+            <parent link="base_link" />
             <child link="${prefix}_wheel" />
             <origin rpy="${pos_r} ${pos_p} ${pos_y}" xyz="${pos_X} ${pos_Y} ${pos_Z}" />
         </joint>
         <gazebo reference="${prefix}_wheel">
-            <selfCollide>false</selfCollide>
+            <selfCollide>true</selfCollide>
             <mu1 value="0.09" />
             <mu2 value="0.09" />

File: ros2_ws/src/warehouse_robot/urdf/robot_parts/piston.xacro (robot description, xacro)
@@ -11,5 +11,5 @@
         </joint>
         <gazebo reference="${prefix}">
-            <selfCollide>false</selfCollide>
+            <selfCollide>true</selfCollide>
             <mu1 value="0.1" />
             <mu2 value="0.1" />

File: ros2_ws/src/warehouse_robot/urdf/robot_parts/traction_wheel.xacro (robot description, xacro)
@@ -3,5 +3,5 @@
     <xacro:macro name="traction_wheel" params="prefix pos_X pos_Y pos_Z pos_r pos_p pos_y axis">
         <joint name="${prefix}_joint" type="continuous">
-            <parent link="carcaca" />
+            <parent link="base_link" />
             <child link="${prefix}" />
             <origin rpy="${pos_r} ${pos_p} ${pos_y}" xyz="${pos_X} ${pos_Y} ${pos_Z}" />
@@ -10,5 +10,5 @@
         </joint>
         <gazebo reference="${prefix}">
-            <selfCollide>false</selfCollide>
+            <selfCollide>true</selfCollide>
             <mu1>1.0</mu1>
             <mu2>1.0</mu2>

File: ros2_ws/src/warehouse_robot/urdf/robot_parts/tray.xacro (robot description, xacro)
@@ -10,5 +10,5 @@
         </joint>
         <gazebo reference="${prefix}">
-            <selfCollide>false</selfCollide>
+            <selfCollide>true</selfCollide>
             <mu1 value="0.1" />
             <mu2 value="0.1" />

Commit message: piston stability tuning for static condition

File: ros2_ws/src/warehouse_robot/urdf/robot_parts/carcaca.xacro (robot description, xacro)
@@ -26,5 +26,5 @@
         <link name="${base_link}">
             <inertial>
-                <mass value="2.4" />
+                <mass value="10" />
                 <origin rpy="0  0  0" xyz="0  0  0.0118" />
                 <inertia ixx="0.019995" ixy="0.0" ixz="0.0"

File: ros2_ws/src/warehouse_robot/urdf/robot_parts/piston.xacro (robot description, xacro)
@@ -3,13 +3,13 @@
     <xacro:macro name="piston" params="prefix">
         <joint name="joint_${prefix}" type="prismatic">
-            <parent link="base_link" />
+            <parent link="carcaca" />
             <child link="${prefix}" />
-            <dynamics friction="5.0" />
+            <dynamics friction="10.0" />
             <origin rpy="0 0 0" xyz="0 0 0.1318" />
             <axis xyz="0 0 1" />
-            <limit effort="0" lower="0" upper="0.04" velocity="0" />
+            <limit effort="10" lower="0" upper="0.08" velocity="0.8" />
         </joint>
         <gazebo reference="${prefix}">
-            <selfCollide>true</selfCollide>
+            <selfCollide>false</selfCollide>
             <mu1 value="0.1" />
             <mu2 value="0.1" />

File: ros2_ws/src/warehouse_robot/urdf/robot_parts/tray.xacro (robot description, xacro)
@@ -2,5 +2,5 @@
 <robot xmlns:xacro="http://www.ros.org/wiki/xacro">
     <xacro:macro name="tray" params="prefix">
-        <joint name="joint_${prefix}" type="continuous">
+        <joint name="joint_${prefix}" type="fixed">
             <parent link="piston" />
             <child link="${prefix}" />
@@ -10,5 +10,5 @@
         </joint>
         <gazebo reference="${prefix}">
-            <selfCollide>true</selfCollide>
+            <selfCollide>false</selfCollide>
             <mu1 value="0.1" />
             <mu2 value="0.1" />

Commit message: Adjusted model weight and friction values to get shelf to lift and move with robot

File: ros2_ws/src/warehouse_robot/urdf/robot_parts/carcaca.xacro (robot description, xacro)
@@ -4,5 +4,5 @@
         <gazebo reference="${base_link}">
             <selfCollide>true</selfCollide>
-            <mu1 value="0.3" />
+            <mu value="0.3" />
             <mu2 value="0.3" />
             <kp value="1000000.0" />
@@ -26,5 +26,5 @@
         <link name="${base_link}">
             <inertial>
-                <mass value="2.4" />
+                <mass value="5" />
                 <origin rpy="0  0  0" xyz="0  0  0.0118" />
                 <inertia ixx="0.019995" ixy="0.0" ixz="0.0"

File: ros2_ws/src/warehouse_robot/urdf/robot_parts/tray.xacro (robot description, xacro)
@@ -2,5 +2,5 @@
 <robot xmlns:xacro="http://www.ros.org/wiki/xacro">
     <xacro:macro name="tray" params="prefix">
-        <joint name="joint_${prefix}" type="continuous">
+        <joint name="joint_${prefix}" type="fixed">
             <parent link="piston" />
             <child link="${prefix}" />
@@ -11,6 +11,6 @@
         <gazebo reference="${prefix}">
             <selfCollide>true</selfCollide>
-            <mu1 value="0.1" />
-            <mu2 value="0.1" />
+            <mu1 value="5" />
+            <mu2 value="5" />
             <kp value="10000000.0" />
             <kd value="10000" />

Commit message: Updates to get single complete loop working

File: ros2_ws/src/warehouse_robot/urdf/robot_parts/carcaca.xacro (robot description, xacro)
@@ -32,5 +32,5 @@
         <link name="${base_link}">
             <inertial>
-                <mass value="5" />
+                <mass value="6" />
                 <origin rpy="0  0  0" xyz="0  0  0.0118" />
                 <inertia ixx="0.019995" ixy="0.0" ixz="0.0"

File: ros2_ws/src/warehouse_robot/urdf/sensors/rplidar.xacro (robot description, xacro)
@@ -40,5 +40,5 @@
             </scan>
             <range>
-                <min>0.8</min>
+                <min>0.3</min>
                 <max>12</max>
             </range>
